File: PCB/gamerino/gamerino.sch (KiCad schematic (older format))
At the start: 12 parts

Commit message: Update
Parts:
- added C1, C2: 10uF, Capacitor_Tantalum_SMD:CP_EIA-3216-18_Kemet-A, symbol device2:CT
- added C10, C6, C7: 100nF, Capacitor_SMD:C_0603_1608Metric, symbol device:C
- added C3, C4: 18pF C0G, Capacitor_SMD:C_0402_1005Metric, symbol device:C
- added C5, C8, C9: 1uF, Capacitor_SMD:C_0603_1608Metric, symbol device:C
- added D1: GREEN, LED_SMD:LED_0603_1608Metric, symbol device:LED
- added F1: 500mA, Fuse:Fuse_0805_2012Metric, symbol w_device:FUSE
- added J2: LT2, Connector_Molex:Molex_PicoBlade_53047-0310_1x03_P1.25mm_Vertical, symbol conn:CONN_3
- added J3: RT2, Connector_Molex:Molex_PicoBlade_53047-0310_1x03_P1.25mm_Vertical, symbol conn:CONN_3
- added P1: JOY1, symbol conn:CONN_4
- added P2: JOY2, symbol conn:CONN_4
- added P3: ICSP, Connector_PinHeader_2.54mm:PinHeader_2x03_P2.54mm_Vertical, symbol conn:CONN_3X2
- added P4: AUX, Connector_PinSocket_1.00mm:PinSocket_2x08_P1.00mm_Vertical_SMD, symbol conn:CONN_8X2
- added R1, R2: 22R, Resistor_SMD:R_0603_1608Metric, symbol device:R
- added R3, R5, R7: 10K, Resistor_SMD:R_0603_1608Metric, symbol device:R
- added R4: 1K, Resistor_SMD:R_0603_1608Metric, symbol device:R
- added R6, R8, R9: 2.2K, Resistor_SMD:R_0603_1608Metric, symbol device:R
- added SW1: HATSWITCH, gamerino:RKJXS, symbol gamerino:RKJXS
- added SW2, SW3, SW4, SW5: SW_Push, symbol gamerino-rescue:SW_Push-Switch
- added U1: MIC5219-3.3YM5, Package_TO_SOT_SMD:SOT-23-5, symbol microchip5:MIC5219-3.3YM5
- added X1: 16MHz, Crystal:Crystal_SMD_2520-4Pin_2.5x2.0mm, symbol device:CRYSTAL
- J1: renamed from J?; footprint (none) -> te:1981568-1; symbol Connector:USB_B_Micro -> gamerino-rescue:USB_B_Micro-Connector
- SW10, SW11, SW12, SW13, SW14, SW6, SW7, SW8, SW9: renamed from SW?; symbol Switch:SW_Push -> gamerino-rescue:SW_Push-Switch
- U2: renamed from U?; value ATmega32U4-MU -> ATmega32U4-AU; footprint Package_DFN_QFN:QFN-44-1EP_7x7mm_P0.5mm_EP5.2x5.2mm -> Package_QFP:LQFP-44_10x10mm_P0.8mm; symbol MCU_Microchip_ATmega:ATmega32U4-MU -> gamerino-rescue:ATmega32U4-MU-MCU_Microchip_ATmega
- U3: renamed from U?; footprint (none) -> Package_SO:TSSOP-24_4.4x7.8mm_P0.65mm; MPN (none) -> TCA9539PWR; Manufacturer (none) -> TI
Connections:
- net +3V3: now also U2.24 (AVCC), U2.44 (AVCC), C10.2, C2.2, C5.1, C6.1, J2.3 (P3), J3.3 (P3), P1.3 (P3), P2.3 (P3), P3.2, P4.16, R3.2, R4.2, R6.2, R7.2, R8.2, R9.1, U1.5 (OUT)
- net GND: now also SW10.2, SW11.2, SW12.2, SW13.2, SW14.2, SW6.2, SW7.2, SW8.2, SW9.2, U2.5 (UGND), U3.12 (GND), U3.2 (A1), U3.21 (A0), C1.1, C10.1, C2.1, C3.2, C4.2, C5.2, C6.2, C7.1, C8.1, C9.2, D1.1 (K), J2.1 (P1), J3.1 (P1), P1.1 (P1), P2.1 (P1), P3.6, P4.1, R5.1, SW1.C, SW2.1, SW3.1, SW4.1, SW5.1, U1.2 (GND)
- net VBUS: now also U2.2 (UVCC), C9.1, F1.1
- net PE6: now reaches U2.1 (PE6)
- net PE6: now also P4.3
- net MOSI: now reaches U2.10 (PB2)
- net MOSI: now also P3.4
- net MISO: now reaches U2.11 (PB3)
- net MISO: now also P3.1
- net PB7: now reaches U2.12 (PB7)
- net PB7: now also P4.8
- net RESET: now reaches U2.13 (~RESET)
- net RESET: now also P3.5, R3.1
- net XTAL2: now reaches U2.16 (XTAL2)
- net XTAL2: now also C4.1, X1.1
- net XTAL1: now reaches U2.17 (XTAL1)
- net XTAL1: now also C3.1, X1.2
- net SDA: now reaches U2.18 (PD0)
- net SDA: now also U3.23 (SDA), R8.1
- net SCL: now reaches U2.19 (PD1)
- net SCL: now also U3.22 (SCL), R6.1
- net PD2: now reaches U2.20 (PD2)
- net PD2: now also P4.15
- net PD3: now reaches U2.21 (PD3)
- net PD3: now also P4.13
- net PD5: now reaches U2.22 (PD5)
- net PD5: now also P4.9
- net PD4: now reaches U2.25 (PD4)
- net PD4: now also P4.11
- net PD6: now reaches U2.26 (PD6)
- net PD6: now also P4.7
- net PD7: now reaches U2.27 (PD7)
- net PD7: now also P4.5
- net PB4: now reaches U2.28 (PB4)
- net PB4: now also P4.14
- net PB5: now reaches U2.29 (PB5)
- net PB5: now also P4.12
- net at U2.3 (D-): now also R2.1; no longer J1.2 (D-)
- net PB6: now reaches U2.30 (PB6)
- net PB6: now also P4.10
- net PC6: now reaches U2.31 (PC6)
- net PC6: now also P4.4
- net PC7: now reaches U2.32 (PC7)
- net PC7: now also P4.2
- net at U2.33 (~HWB~/PE2): now also R5.2
- net RT2: now reaches U2.36 (PF7)
- net RT2: now also J3.2 (PM), SW5.2
- net LT2: now reaches U2.37 (PF6)
- net LT2: now also J2.2 (PM), SW3.2
- net J2Y: now reaches U2.38 (PF5)
- net J2Y: now also P2.2 (P2)
- net J2X: now reaches U2.39 (PF4)
- net J2X: now also P2.4 (P4)
- net at U2.4 (D+): now also R1.1; no longer J1.3 (D+)
- net J1Y: now reaches U2.40 (PF1)
- net J1Y: now also P1.2 (P2)
- net J1X: now reaches U2.41 (PF0)
- net J1X: now also P1.4 (P4)
- net at U2.42 (AREF): now also C7.2
- net at U2.6 (UCAP): now also C8.2
- net IRQ: now reaches U2.8 (PB0)
- net IRQ: now also U3.1 (INT), R9.2
- net SCK: now reaches U2.9 (PB1)
- net SCK: now also P3.3
- net B: now reaches U3.10 (P06)
- net B: now also SW12.1
- net A: now reaches U3.11 (P07)
- net A: now also SW13.1
- net Y: now reaches U3.13 (P10)
- net Y: now also SW14.1
- net HP: now reaches U3.14 (P11)
- net HP: now also SW1.P
- net HW: now reaches U3.15 (P12)
- net HW: now also SW1.4
- net HN: now reaches U3.16 (P13)
- net HN: now also SW1.1
- net HE: now reaches U3.17 (P14)
- net HE: now also SW1.2
- net HS: now reaches U3.18 (P15)
- net HS: now also SW1.3
- net LT1: now reaches U3.19 (P16)
- net LT1: now also SW2.2
- net RT1: now reaches U3.20 (P17)
- net RT1: now also SW4.2
- net at U3.3 (RESET): now also R7.1
- net SELECT: now reaches U3.4 (P00)
- net SELECT: now also SW6.1
- net START: now reaches U3.5 (P01)
- net START: now also SW7.1
- net CLEAR: now reaches U3.6 (P02)
- net CLEAR: now also SW8.1
- net HOME: now reaches U3.7 (P03)
- net HOME: now also SW9.1
- net OPTS: now reaches U3.8 (P04)
- net X: now reaches U3.9 (P05)
- net X: now also SW11.1
- net OPTIONS: now reaches SW10.1
- new net: J1.2 (D-), R2.2
- new net: J1.3 (D+), R1.2
- new net: C1.2, F1.2, U1.1 (IN), U1.3 (EN)
- new net: D1.2 (A), R4.1
- no-connect marks 1 -> 3
Other:
- note added: "CROSS"
- note added: "SPARE"
- note added: "TRIGGERS"
- moved on the sheet: J1, SW10, SW11, SW12, SW13, SW14, SW6, SW7, SW8, SW9, U2, U3

Commit message: Update
Parts:
- P1, P2: footprint (none) -> gamerino:52746-0471; MPN (none) -> 52746-0471; Manufacturer (none) -> Molex
Other:
- moved on the sheet: J2, P4
Changed lines of the file:
@@
 P 5200 4350
 F 0 "#PWR016" H 5200 4200 50  0001 C CNN
-F 1 "VBUS" V 5250 4500 50  0000 L CNN
+F 1 "VBUS" V 5050 4350 50  0000 C CNN
 F 2 "" H 5200 4350 50  0001 C CNN
 F 3 "" H 5200 4350 50  0001 C CNN
@@
 F 0 "P1" H 4100 7700 50  0000 C CNN
 F 1 "JOY1" H 4100 7800 50  0000 C CNN
-F 2 "" H 4225 8125 50  0001 C CNN
+F 2 "gamerino:52746-0471" H 4225 8125 50  0001 C CNN
 F 3 "" H 4225 8125 50  0001 C CNN
+F 4 "52746-0471" H 4225 8125 50  0001 C CNN "MPN"
+F 5 "Molex" H 4225 8125 50  0001 C CNN "Manufacturer"
 	1    4225 8125
 	1    0    0    1
@@
 F 0 "P2" H 4400 8600 50  0000 L CNN
 F 1 "JOY2" H 4400 8700 50  0000 L CNN
-F 2 "" H 4225 8700 50  0001 C CNN
+F 2 "gamerino:52746-0471" H 4225 8700 50  0001 C CNN
 F 3 "" H 4225 8700 50  0001 C CNN
+F 4 "52746-0471" H 4225 8700 50  0001 C CNN "MPN"
+F 5 "Molex" H 4225 8700 50  0001 C CNN "Manufacturer"
 	1    4225 8700
 	1    0    0    1
@@
 	7825 9925 7600 9925
 Wire Wire Line
-	7600 8350 7825 8350
+	7600 8075 7825 8075
 $Comp
 L gamerino-rescue:GND-power #PWR026
@@
 P 4825 5150
 F 0 "#PWR014" H 4825 4900 50  0001 C CNN
-F 1 "GND" H 4830 4977 50  0000 C CNN
+F 1 "GND" H 4850 4950 50  0000 C CNN
 F 2 "" H 4825 5150 50  0001 C CNN
 F 3 "" H 4825 5150 50  0001 C CNN
@@
 $EndComp
 Wire Wire Line
-	4825 4850 4825 4150
-Wire Wire Line
 	4825 4150 4975 4150
-Connection ~ 4825 4850
 Wire Wire Line
 	5375 4150 5475 4150
@@
 Text Label 10500 4950 0    50   ~ 0
 RT1
-Text Label 7600 8350 2    50   ~ 0
+Text Label 7600 8075 2    50   ~ 0
 LT2
 Text Label 7600 9925 2    50   ~ 0
@@
 L conn:CONN_8X2 P4
 U 1 1 60F69BD5
-P 6075 8400
-F 0 "P4" H 6050 7800 47  0000 C CNN
-F 1 "AUX" H 6050 7900 50  0000 C CNN
-F 2 "Connector_PinSocket_1.00mm:PinSocket_2x08_P1.00mm_Vertical_SMD" H 6075 8400 50  0001 C CNN
-F 3 "" H 6075 8400 50  0001 C CNN
-	1    6075 8400
+P 6075 8325
+F 0 "P4" H 6050 7725 47  0000 C CNN
+F 1 "AUX" H 6050 7825 50  0000 C CNN
+F 2 "Connector_PinSocket_1.00mm:PinSocket_2x08_P1.00mm_Vertical_SMD" H 6075 8325 50  0001 C CNN
+F 3 "" H 6075 8325 50  0001 C CNN
+	1    6075 8325
 	-1   0    0    1
 $EndComp
@@
 PD3
 Wire Wire Line
-	6475 8250 6875 8250
-Text Label 6875 8250 0    50   ~ 0
+	6475 8175 6875 8175
+Text Label 6875 8175 0    50   ~ 0
 PD4
 Wire Wire Line
-	6475 8350 6875 8350
-Text Label 6875 8350 0    50   ~ 0
+	6475 8275 6875 8275
+Text Label 6875 8275 0    50   ~ 0
 PD5
 Wire Wire Line
-	6475 8450 6875 8450
-Text Label 6875 8450 0    50   ~ 0
+	6475 8375 6875 8375
+Text Label 6875 8375 0    50   ~ 0
 PD6
 Wire Wire Line
-	6475 8550 6875 8550
-Text Label 6875 8550 0    50   ~ 0
+	6475 8475 6875 8475
+Text Label 6875 8475 0    50   ~ 0
 PD7
 Wire Wire Line
-	6475 8050 6875 8050
-Text Label 6875 8050 0    50   ~ 0
+	6475 7975 6875 7975
+Text Label 6875 7975 0    50   ~ 0
 PD2
 Wire Wire Line
-	6475 8150 6875 8150
-Text Label 6875 8150 0    50   ~ 0
+	6475 8075 6875 8075
+Text Label 6875 8075 0    50   ~ 0
 PD3
 Text Label 7075 4250 0    50   ~ 0
@@
 Wire Wire Line
 	6675 3850 7075 3850
-Text Label 5275 8450 2    50   ~ 0
+Text Label 5275 8375 2    50   ~ 0
 PB7
 Wire Wire Line
-	5675 8450 5275 8450
-Text Label 5275 8350 2    50   ~ 0
+	5675 8375 5275 8375
+Text Label 5275 8275 2    50   ~ 0
 PB6
 Wire Wire Line
-	5675 8350 5275 8350
-Text Label 5275 8250 2    50   ~ 0
+	5675 8275 5275 8275
+Text Label 5275 8175 2    50   ~ 0
 PB5
 Wire Wire Line
-	5675 8250 5275 8250
-Text Label 5275 8150 2    50   ~ 0
+	5675 8175 5275 8175
+Text Label 5275 8075 2    50   ~ 0
 PB4
 Wire Wire Line
-	5675 8150 5275 8150
+	5675 8075 5275 8075
 $Comp
 L gamerino-rescue:+3.3V-power #PWR017
@@
 P 5500 7825
 F 0 "#PWR017" H 5500 7675 50  0001 C CNN
-F 1 "+3.3V" H 5425 7900 50  0000 R CNN
+F 1 "+3.3V" H 5550 8050 50  0000 C CNN
 F 2 "" H 5500 7825 50  0001 C CNN
 F 3 "" H 5500 7825 50  0001 C CNN
@@
 $EndComp
 Wire Wire Line
-	5500 7825 5500 8050
-Wire Wire Line
-	5500 8050 5675 8050
-Wire Wire Line
-	6475 8750 6675 8750
-Wire Wire Line
-	6675 8750 6675 9000
+	5500 7825 5500 7975
+Wire Wire Line
+	5500 7975 5675 7975
+Wire Wire Line
+	6475 8675 6675 8675
+Wire Wire Line
+	6675 8675 6675 8925
 $Comp
 L gamerino-rescue:GND-power #PWR022
 U 1 1 6104C98A
-P 6675 9000
-F 0 "#PWR022" H 6675 8750 50  0001 C CNN
-F 1 "GND" H 6700 8775 50  0000 C CNN
-F 2 "" H 6675 9000 50  0001 C CNN
-F 3 "" H 6675 9000 50  0001 C CNN
-	1    6675 9000
-	1    0    0    -1
-$EndComp
-Wire Wire Line
-	5675 8650 5275 8650
-Text Label 5275 8650 2    50   ~ 0
+P 6675 8925
+F 0 "#PWR022" H 6675 8675 50  0001 C CNN
+F 1 "GND" H 6700 8700 50  0000 C CNN
+F 2 "" H 6675 8925 50  0001 C CNN
+F 3 "" H 6675 8925 50  0001 C CNN
+	1    6675 8925
+	1    0    0    -1
+$EndComp
+Wire Wire Line
+	5675 8575 5275 8575
+Text Label 5275 8575 2    50   ~ 0
 PC6
 Wire Wire Line
-	5675 8750 5275 8750
-Text Label 5275 8750 2    50   ~ 0
+	5675 8675 5275 8675
+Text Label 5275 8675 2    50   ~ 0
 PC7
-NoConn ~ 5675 8550
-Wire Wire Line
-	6475 8650 6875 8650
-Text Label 6875 8650 0    50   ~ 0
+NoConn ~ 5675 8475
+Wire Wire Line
+	6475 8575 6875 8575
+Text Label 6875 8575 0    50   ~ 0
 PE6
 Wire Wire Line
@@
 L gamerino-rescue:+3.3V-power #PWR023
 U 1 1 6116AC53
-P 7825 8000
-F 0 "#PWR023" H 7825 7850 50  0001 C CNN
-F 1 "+3.3V" H 7800 8200 50  0000 C CNN
-F 2 "" H 7825 8000 50  0001 C CNN
-F 3 "" H 7825 8000 50  0001 C CNN
-	1    7825 8000
+P 7825 7725
+F 0 "#PWR023" H 7825 7575 50  0001 C CNN
+F 1 "+3.3V" H 7800 7925 50  0000 C CNN
+F 2 "" H 7825 7725 50  0001 C CNN
+F 3 "" H 7825 7725 50  0001 C CNN
+	1    7825 7725
 	-1   0    0    -1
 $EndComp
@@
 L gamerino-rescue:GND-power #PWR024
 U 1 1 6116B2BE
-P 7825 8775
-F 0 "#PWR024" H 7825 8525 50  0001 C CNN
-F 1 "GND" H 7800 8550 50  0000 C CNN
-F 2 "" H 7825 8775 50  0001 C CNN
-F 3 "" H 7825 8775 50  0001 C CNN
-	1    7825 8775
-	-1   0    0    -1
-$EndComp
-Wire Wire Line
-	7825 8000 7825 8250
-Wire Wire Line
-	7825 8450 7825 8775
+P 7825 8500
+F 0 "#PWR024" H 7825 8250 50  0001 C CNN
+F 1 "GND" H 7800 8275 50  0000 C CNN
+F 2 "" H 7825 8500 50  0001 C CNN
+F 3 "" H 7825 8500 50  0001 C CNN
+	1    7825 8500
+	-1   0    0    -1
+$EndComp
+Wire Wire Line
+	7825 7725 7825 7975
+Wire Wire Line
+	7825 8175 7825 8500
 $Comp
 L conn:CONN_3 J2
 U 1 1 6116B2CB
-P 8175 8350
-F 0 "J2" H 8050 8000 50  0000 C CNN
-F 1 "LT2" H 8050 8100 50  0000 C CNN
-F 2 "Connector_Molex:Molex_PicoBlade_53047-0310_1x03_P1.25mm_Vertical" H 8175 8350 50  0001 C CNN
-F 3 "" H 8175 8350 50  0001 C CNN
-F 4 "53047-0310" H 8175 8350 50  0001 C CNN "MPN"
-F 5 "Molex" H 8175 8350 50  0001 C CNN "Manufacturer"
-	1    8175 8350
+P 8175 8075
+F 0 "J2" H 8050 7725 50  0000 C CNN
+F 1 "LT2" H 8050 7825 50  0000 C CNN
+F 2 "Connector_Molex:Molex_PicoBlade_53047-0310_1x03_P1.25mm_Vertical" H 8175 8075 50  0001 C CNN
+F 3 "" H 8175 8075 50  0001 C CNN
+F 4 "53047-0310" H 8175 8075 50  0001 C CNN "MPN"
+F 5 "Molex" H 8175 8075 50  0001 C CNN "Manufacturer"
+	1    8175 8075
 	1    0    0    1
 $EndComp
+$Comp
+L gamerino-rescue:GND-power #PWR?
+U 1 1 60A7A8F7
+P 4825 4325
+F 0 "#PWR?" H 4825 4075 50  0001 C CNN
+F 1 "GND" H 4700 4300 50  0000 R CNN
+F 2 "" H 4825 4325 50  0001 C CNN
+F 3 "" H 4825 4325 50  0001 C CNN
+	1    4825 4325
+	1    0    0    -1
+$EndComp
+Wire Wire Line
+	4825 4325 4825 4150
 $EndSCHEMATC
