File: PCB/gamerino.sch (KiCad schematic (older format))
At the start: 46 parts, among them J1 USB_B_Micro, J2 LT2, J3 RT2, P1 JOY1, P2 JOY2, P3 ICSP, P4 AUX, SW1 HATSWITCH, SW10 SW_Push, SW11 SW_Push, SW12 SW_Push, SW13 SW_Push, SW14 SW_Push, SW2 SW_Push, SW3 SW_Push, SW4 SW_Push, SW5 SW_Push, SW6 SW_Push, SW7 SW_Push, SW8 SW_Push, SW9 SW_Push, U1 MIC5219-3.3YM5, U2 ATmega32U4-AU, U3 TCA9539, X1 16MHz

Commit message: Update
Parts:
- C1, C2: symbol device2:CT -> gamerino-rescue:CT-device2
- C10, C3, C4, C5, C6, C7, C8, C9: symbol device:C -> gamerino-rescue:C-device
- D1: symbol device:LED -> gamerino-rescue:LED-device
- F1: symbol w_device:FUSE -> gamerino-rescue:FUSE-w_device
- J1: footprint te:1981568-1 -> gamerino:TE_1981568-1; MPN (none) -> 1981568-1; Manufacturer (none) -> TE
- J2, J3: symbol conn:CONN_3 -> gamerino-rescue:CONN_3-conn
- P1, P2: symbol conn:CONN_4 -> gamerino-rescue:CONN_4-conn
- P3: symbol conn:CONN_3X2 -> gamerino-rescue:CONN_3X2-conn
- P4: symbol conn:CONN_8X2 -> gamerino-rescue:CONN_8X2-conn
- R1, R2, R3, R4, R5, R6, R7, R8, R9: symbol device:R -> gamerino-rescue:R-device
- SW10, SW11, SW12, SW13, SW14, SW6, SW7, SW8, SW9: footprint (none) -> gamerino:B3FS-1052; MPN (none) -> B3FS-1052; Manufacturer (none) -> Omron
- SW2, SW3, SW4, SW5: footprint (none) -> gamerino:B3F-3155; MPN (none) -> B3F-3152; Manufacturer (none) -> Omron
- U1: symbol microchip5:MIC5219-3.3YM5 -> gamerino-rescue:MIC5219-3.3YM5-microchip5; MPN (none) -> MIC5219-3.3YM5; Manufacturer (none) -> Micrel
- U2: value ATmega32U4-AU -> ATmega32U4; MPN (none) -> ATmega32U4-AU; Manufacturer (none) -> Atmel
- X1: symbol device:CRYSTAL -> gamerino-rescue:CRYSTAL-device; Manufacturer (none) -> Murata
Changed lines of the file:
@@
 P 6075 5050
 F 0 "U2" H 5625 6825 50  0000 C CNN
-F 1 "ATmega32U4-AU" H 6550 6825 50  0000 C CNN
+F 1 "ATmega32U4" H 6550 6825 50  0000 C CNN
 F 2 "Package_QFP:LQFP-44_10x10mm_P0.8mm" H 6075 5050 50  0001 C CIN
 F 3 "http://ww1.microchip.com/downloads/en/DeviceDoc/Atmel-7766-8-bit-AVR-ATmega16U4-32U4_Datasheet.pdf" H 6075 5050 50  0001 C CNN
+F 4 "ATmega32U4-AU" H 6075 5050 50  0001 C CNN "MPN"
+F 5 "Atmel" H 6075 5050 50  0001 C CNN "Manufacturer"
 	1    6075 5050
 	1    0    0    -1
@@
 F 0 "SW6" H 14500 1900 50  0000 C CNN
 F 1 "SW_Push" H 14500 1800 50  0000 C CNN
-F 2 "" H 14500 1800 50  0001 C CNN
+F 2 "gamerino:B3FS-1052" H 14500 1800 50  0001 C CNN
 F 3 "~" H 14500 1800 50  0001 C CNN
+F 4 "B3FS-1052" H 14500 1600 50  0001 C CNN "MPN"
+F 5 "Omron" H 14500 1600 50  0001 C CNN "Manufacturer"
 	1    14500 1600
 	1    0    0    -1
@@
 F 0 "SW7" H 14500 2300 50  0000 C CNN
 F 1 "SW_Push" H 14500 2200 50  0000 C CNN
-F 2 "" H 14500 2175 50  0001 C CNN
+F 2 "gamerino:B3FS-1052" H 14500 2175 50  0001 C CNN
 F 3 "~" H 14500 2175 50  0001 C CNN
+F 4 "B3FS-1052" H 14500 1975 50  0001 C CNN "MPN"
+F 5 "Omron" H 14500 1975 50  0001 C CNN "Manufacturer"
 	1    14500 1975
 	1    0    0    -1
@@
 F 0 "SW8" H 14500 2650 50  0000 C CNN
 F 1 "SW_Push" H 14500 2550 50  0000 C CNN
-F 2 "" H 14500 2550 50  0001 C CNN
+F 2 "gamerino:B3FS-1052" H 14500 2550 50  0001 C CNN
 F 3 "~" H 14500 2550 50  0001 C CNN
+F 4 "B3FS-1052" H 14500 2350 50  0001 C CNN "MPN"
+F 5 "Omron" H 14500 2350 50  0001 C CNN "Manufacturer"
 	1    14500 2350
 	1    0    0    -1
@@
 F 0 "SW9" H 14500 3050 50  0000 C CNN
 F 1 "SW_Push" H 14500 2950 50  0000 C CNN
-F 2 "" H 14500 2925 50  0001 C CNN
+F 2 "gamerino:B3FS-1052" H 14500 2925 50  0001 C CNN
 F 3 "~" H 14500 2925 50  0001 C CNN
+F 4 "B3FS-1052" H 14500 2725 50  0001 C CNN "MPN"
+F 5 "Omron" H 14500 2725 50  0001 C CNN "Manufacturer"
 	1    14500 2725
 	1    0    0    -1
@@
 F 0 "SW10" H 14500 3400 50  0000 C CNN
 F 1 "SW_Push" H 14500 3300 50  0000 C CNN
-F 2 "" H 14500 3300 50  0001 C CNN
+F 2 "gamerino:B3FS-1052" H 14500 3300 50  0001 C CNN
 F 3 "~" H 14500 3300 50  0001 C CNN
+F 4 "B3FS-1052" H 14500 3100 50  0001 C CNN "MPN"
+F 5 "Omron" H 14500 3100 50  0001 C CNN "Manufacturer"
 	1    14500 3100
 	1    0    0    -1
@@
 F 0 "SW11" H 14500 4100 50  0000 C CNN
 F 1 "SW_Push" H 14500 4000 50  0000 C CNN
-F 2 "" H 14500 3975 50  0001 C CNN
+F 2 "gamerino:B3FS-1052" H 14500 3975 50  0001 C CNN
 F 3 "~" H 14500 3975 50  0001 C CNN
+F 4 "B3FS-1052" H 14500 3775 50  0001 C CNN "MPN"
+F 5 "Omron" H 14500 3775 50  0001 C CNN "Manufacturer"
 	1    14500 3775
 	1    0    0    -1
@@
 F 0 "SW12" H 14500 4450 50  0000 C CNN
 F 1 "SW_Push" H 14500 4350 50  0000 C CNN
-F 2 "" H 14500 4350 50  0001 C CNN
+F 2 "gamerino:B3FS-1052" H 14500 4350 50  0001 C CNN
 F 3 "~" H 14500 4350 50  0001 C CNN
+F 4 "B3FS-1052" H 14500 4150 50  0001 C CNN "MPN"
+F 5 "Omron" H 14500 4150 50  0001 C CNN "Manufacturer"
 	1    14500 4150
 	1    0    0    -1
@@
 F 0 "SW13" H 14500 4850 50  0000 C CNN
 F 1 "SW_Push" H 14500 4750 50  0000 C CNN
-F 2 "" H 14500 4725 50  0001 C CNN
+F 2 "gamerino:B3FS-1052" H 14500 4725 50  0001 C CNN
 F 3 "~" H 14500 4725 50  0001 C CNN
+F 4 "B3FS-1052" H 14500 4525 50  0001 C CNN "MPN"
+F 5 "Omron" H 14500 4525 50  0001 C CNN "Manufacturer"
 	1    14500 4525
 	1    0    0    -1
@@
 F 0 "SW14" H 14500 5200 50  0000 C CNN
 F 1 "SW_Push" H 14500 5100 50  0000 C CNN
-F 2 "" H 14500 5100 50  0001 C CNN
+F 2 "gamerino:B3FS-1052" H 14500 5100 50  0001 C CNN
 F 3 "~" H 14500 5100 50  0001 C CNN
+F 4 "B3FS-1052" H 14500 4900 50  0001 C CNN "MPN"
+F 5 "Omron" H 14500 4900 50  0001 C CNN "Manufacturer"
 	1    14500 4900
 	1    0    0    -1
@@
 F 0 "J1" H 3800 5050 50  0000 C CNN
 F 1 "USB_B_Micro" H 3800 4950 50  0000 C CNN
-F 2 "te:1981568-1" H 3875 4500 50  0001 C CNN
+F 2 "gamerino:TE_1981568-1" H 3875 4500 50  0001 C CNN
 F 3 "~" H 3875 4500 50  0001 C CNN
+F 4 "1981568-1" H 3725 4550 50  0001 C CNN "MPN"
+F 5 "TE" H 3725 4550 50  0001 C CNN "Manufacturer"
 	1    3725 4550
 	1    0    0    -1
@@
 	8325 4150 8500 4150
 $Comp
-L device:R R7
+L gamerino-rescue:R-device R7
 U 1 1 60A6DF34
 P 8725 3550
@@
 SPARE
 $Comp
-L device:CRYSTAL X1
+L gamerino-rescue:CRYSTAL-device X1
 U 1 1 60A7134E
 P 4325 6125
@@
 F 3 "" H 4325 6125 60  0001 C CNN
 F 4 "XRCHA16M000F0A01R0" V 4325 6125 50  0001 C CNN "MPN"
+F 5 "Murata" H 4325 6125 50  0001 C CNN "Manufacturer"
 	1    4325 6125
 	0    -1   -1   0
 $EndComp
 $Comp
-L device:C C4
+L gamerino-rescue:C-device C4
 U 1 1 60A7270D
 P 3975 6425
@@
 $EndComp
 $Comp
-L device:C C3
+L gamerino-rescue:C-device C3
 U 1 1 60A72D0E
 P 3975 5825
@@
 	6675 6450 7075 6450
 $Comp
-L conn:CONN_4 P1
+L gamerino-rescue:CONN_4-conn P1
 U 1 1 60A872FE
 P 4225 8125
@@
 $EndComp
 $Comp
-L conn:CONN_4 P2
+L gamerino-rescue:CONN_4-conn P2
 U 1 1 60A87A63
 P 4225 8700
@@
 F 0 "SW2" H 14450 5900 50  0000 C CNN
 F 1 "SW_Push" H 14450 5800 50  0000 C CNN
-F 2 "" H 14450 5800 50  0001 C CNN
+F 2 "gamerino:B3F-3155" H 14450 5800 50  0001 C CNN
 F 3 "~" H 14450 5800 50  0001 C CNN
+F 4 "B3F-3152" H 14450 5600 50  0001 C CNN "MPN"
+F 5 "Omron" H 14450 5600 50  0001 C CNN "Manufacturer"
 	1    14450 5600
 	-1   0    0    -1
@@
 F 0 "SW3" H 14450 6300 50  0000 C CNN
 F 1 "SW_Push" H 14450 6200 50  0000 C CNN
-F 2 "" H 14450 6175 50  0001 C CNN
+F 2 "gamerino:B3F-3155" H 14450 6175 50  0001 C CNN
 F 3 "~" H 14450 6175 50  0001 C CNN
+F 4 "B3F-3152" H 14450 5975 50  0001 C CNN "MPN"
+F 5 "Omron" H 14450 5975 50  0001 C CNN "Manufacturer"
 	1    14450 5975
 	-1   0    0    -1
@@
 F 0 "SW4" H 14450 6650 50  0000 C CNN
 F 1 "SW_Push" H 14450 6550 50  0000 C CNN
-F 2 "" H 14450 6550 50  0001 C CNN
+F 2 "gamerino:B3F-3155" H 14450 6550 50  0001 C CNN
 F 3 "~" H 14450 6550 50  0001 C CNN
+F 4 "B3F-3152" H 14450 6350 50  0001 C CNN "MPN"
+F 5 "Omron" H 14450 6350 50  0001 C CNN "Manufacturer"
 	1    14450 6350
 	-1   0    0    -1
@@
 F 0 "SW5" H 14450 7050 50  0000 C CNN
 F 1 "SW_Push" H 14450 6950 50  0000 C CNN
-F 2 "" H 14450 6925 50  0001 C CNN
+F 2 "gamerino:B3F-3155" H 14450 6925 50  0001 C CNN
 F 3 "~" H 14450 6925 50  0001 C CNN
+F 4 "B3F-3152" H 14450 6725 50  0001 C CNN "MPN"
+F 5 "Omron" H 14450 6725 50  0001 C CNN "Manufacturer"
 	1    14450 6725
 	-1   0    0    -1
@@
 	10325 4950 10500 4950
 $Comp
-L conn:CONN_3X2 P3
+L gamerino-rescue:CONN_3X2-conn P3
 U 1 1 60BFF64E
 P 4225 9975
@@
 $EndComp
 $Comp
-L device:C C10
+L gamerino-rescue:C-device C10
 U 1 1 60C02BBD
 P 10225 3100
@@
 	6075 7025 6075 7225
 $Comp
-L device:C C8
+L gamerino-rescue:C-device C8
 U 1 1 60A8B583
 P 5175 4850
@@
 	6175 3125 6075 3125
 $Comp
-L device:C C7
+L gamerino-rescue:C-device C7
 U 1 1 60AF196A
 P 5175 4150
@@
 	6675 5650 7175 5650
 $Comp
-L device:C C5
+L gamerino-rescue:C-device C5
 U 1 1 60C4C88C
 P 4050 1900
@@
 $EndComp
 $Comp
-L device:R R6
+L gamerino-rescue:R-device R6
 U 1 1 60C93238
 P 8500 4625
@@
 $EndComp
 $Comp
-L device:R R8
+L gamerino-rescue:R-device R8
 U 1 1 60C9CA74
 P 8725 4625
@@
 	8500 4950 8500 4875
 $Comp
-L device:R R9
+L gamerino-rescue:R-device R9
 U 1 1 60CE92FE
 P 9225 3050
@@
 	8375 3550 8475 3550
 $Comp
-L device:R R1
+L gamerino-rescue:R-device R1
 U 1 1 60D0903C
 P 4425 4550
@@
 	4675 4550 5475 4550
 $Comp
-L device:R R2
+L gamerino-rescue:R-device R2
 U 1 1 60D0975D
 P 4425 4650
@@
 	5975 3000 5975 3125
 $Comp
-L device:C C9
+L gamerino-rescue:C-device C9
 U 1 1 60D1E38F
 P 5475 3125
@@
 	5125 3125 5275 3125
 $Comp
-L microchip5:MIC5219-3.3YM5 U1
+L gamerino-rescue:MIC5219-3.3YM5-microchip5 U1
 U 1 1 60D540E0
 P 2850 1725
@@
 F 2 "Package_TO_SOT_SMD:SOT-23-5" H 2525 1600 50  0001 C CNN
 F 3 "" H 2525 1600 50  0001 C CNN
+F 4 "MIC5219-3.3YM5" H 2850 1725 50  0001 C CNN "MPN"
+F 5 "Micrel" H 2850 1725 50  0001 C CNN "Manufacturer"
 	1    2850 1725
 	1    0    0    -1
@@
 $EndComp
 $Comp
-L w_device:FUSE F1
+L gamerino-rescue:FUSE-w_device F1
 U 1 1 60D54F5D
 P 1750 1600
@@
 $EndComp
 $Comp
-L device2:CT C1
+L gamerino-rescue:CT-device2 C1
 U 1 1 60D561C8
 P 2000 1900
@@
 	1325 1600 1600 1600
 $Comp
-L device2:CT C2
+L gamerino-rescue:CT-device2 C2
 U 1 1 60DA3854
 P 3475 1900
@@
 $EndComp
 $Comp
-L device:C C6
+L gamerino-rescue:C-device C6
 U 1 1 60C4B9EB
 P 4550 1900
@@
 Connection ~ 4050 2200
 $Comp
-L device:R R4
+L gamerino-rescue:R-device R4
 U 1 1 60E4EB67
 P 5000 1600
@@
 	4550 1600 4750 1600
 $Comp
-L device:LED D1
+L gamerino-rescue:LED-device D1
 U 1 1 60E6894D
 P 5575 1600
@@
 	5775 1600 5975 1600
 $Comp
-L device:R R3
+L gamerino-rescue:R-device R3
 U 1 1 60ED079A
 P 4550 3050
@@
 RT2
 $Comp
-L conn:CONN_8X2 P4
+L gamerino-rescue:CONN_8X2-conn P4
 U 1 1 60F69BD5
 P 6075 8325
@@
 $EndComp
 $Comp
-L device:R R5
+L gamerino-rescue:R-device R5
 U 1 1 60C40C2E
 P 7425 5650
@@
 	13900 4150 14300 4150
 $Comp
-L conn:CONN_3 J3
+L gamerino-rescue:CONN_3-conn J3
 U 1 1 61121A56
 P 8175 9925
@@
 	7825 8175 7825 8500
 $Comp
-L conn:CONN_3 J2
+L gamerino-rescue:CONN_3-conn J2
 U 1 1 6116B2CB
 P 8175 8075
@@
 $EndComp
 $Comp
-L gamerino-rescue:GND-power #PWR?
+L gamerino-rescue:GND-power #PWR0101
 U 1 1 60A7A8F7
 P 4825 4325
-F 0 "#PWR?" H 4825 4075 50  0001 C CNN
+F 0 "#PWR0101" H 4825 4075 50  0001 C CNN
 F 1 "GND" H 4700 4300 50  0000 R CNN
 F 2 "" H 4825 4325 50  0001 C CNN

Commit message: Update
Parts:
- J2, J3: footprint Connector_Molex:Molex_PicoBlade_53047-0310_1x03_P1.25mm_Vertical -> gamerino:53398-0371
Connections:
- net CLEAR: no longer SW8.1
- new net BACK: SW8.1
Changed lines of the file:
@@
 START
 Text Label 13900 2350 2    50   ~ 0
-CLEAR
+BACK
 Text Label 13900 2725 2    50   ~ 0
 HOME
@@
 F 0 "J3" H 8050 9550 50  0000 C CNN
 F 1 "RT2" H 8050 9650 50  0000 C CNN
-F 2 "Connector_Molex:Molex_PicoBlade_53047-0310_1x03_P1.25mm_Vertical" H 8175 9925 50  0001 C CNN
+F 2 "gamerino:53398-0371" H 8175 9925 50  0001 C CNN
 F 3 "" H 8175 9925 50  0001 C CNN
 F 4 "53047-0310" H 8175 9925 50  0001 C CNN "MPN"
@@
 F 0 "J2" H 8050 7725 50  0000 C CNN
 F 1 "LT2" H 8050 7825 50  0000 C CNN
-F 2 "Connector_Molex:Molex_PicoBlade_53047-0310_1x03_P1.25mm_Vertical" H 8175 8075 50  0001 C CNN
+F 2 "gamerino:53398-0371" H 8175 8075 50  0001 C CNN
 F 3 "" H 8175 8075 50  0001 C CNN
 F 4 "53047-0310" H 8175 8075 50  0001 C CNN "MPN"

Commit message: Update
Parts:
- SW10: value SW_Push -> OPTS
- SW11: value SW_Push -> X; footprint gamerino:B3FS-1052 -> gamerino:TL1220; MPN B3FS-1052 -> TL1220R1BBBNN; Manufacturer Omron -> E-Switch
- SW12: value SW_Push -> B; footprint gamerino:B3FS-1052 -> gamerino:TL1220; MPN B3FS-1052 -> TL1220R1BBBNN; Manufacturer Omron -> E-Switch
- SW13: value SW_Push -> A; footprint gamerino:B3FS-1052 -> gamerino:TL1220; MPN B3FS-1052 -> TL1220R1BBBNN; Manufacturer Omron -> E-Switch
- SW14: value SW_Push -> Y; footprint gamerino:B3FS-1052 -> gamerino:TL1220; MPN B3FS-1052 -> TL1220R1BBBNN; Manufacturer Omron -> E-Switch
- SW2: value SW_Push -> LT1; footprint gamerino:B3F-3155 -> gamerino:TL6215-R; MPN B3F-3152 -> TL6215RF200NDK; Manufacturer Omron -> E-Switch
- SW3: value SW_Push -> LT2; footprint gamerino:B3F-3155 -> gamerino:TL6215-R; MPN B3F-3152 -> TL6215RF200NDK; Manufacturer Omron -> E-Switch
- SW4: value SW_Push -> RT1; footprint gamerino:B3F-3155 -> gamerino:TL6215-R; MPN B3F-3152 -> TL6215RF200NDK; Manufacturer Omron -> E-Switch
- SW5: value SW_Push -> RT2; footprint gamerino:B3F-3155 -> gamerino:TL6215-R; MPN B3F-3152 -> TL6215RF200NDK; Manufacturer Omron -> E-Switch
- SW6: value SW_Push -> SEL
- SW7: value SW_Push -> START
- SW8: value SW_Push -> BACK
- SW9: value SW_Push -> HOME; footprint gamerino:B3FS-1052 -> gamerino:TL1220; MPN B3FS-1052 -> TL1220R3BBBNN; Manufacturer Omron -> E-Switch
Changed lines of the file:
@@
 P 14500 1600
 F 0 "SW6" H 14500 1900 50  0000 C CNN
-F 1 "SW_Push" H 14500 1800 50  0000 C CNN
+F 1 "SEL" H 14500 1800 50  0000 C CNN
 F 2 "gamerino:B3FS-1052" H 14500 1800 50  0001 C CNN
 F 3 "~" H 14500 1800 50  0001 C CNN
@@
 P 14500 1975
 F 0 "SW7" H 14500 2300 50  0000 C CNN
-F 1 "SW_Push" H 14500 2200 50  0000 C CNN
+F 1 "START" H 14500 2200 50  0000 C CNN
 F 2 "gamerino:B3FS-1052" H 14500 2175 50  0001 C CNN
 F 3 "~" H 14500 2175 50  0001 C CNN
@@
 P 14500 2350
 F 0 "SW8" H 14500 2650 50  0000 C CNN
-F 1 "SW_Push" H 14500 2550 50  0000 C CNN
+F 1 "BACK" H 14500 2550 50  0000 C CNN
 F 2 "gamerino:B3FS-1052" H 14500 2550 50  0001 C CNN
 F 3 "~" H 14500 2550 50  0001 C CNN
@@
 P 14500 2725
 F 0 "SW9" H 14500 3050 50  0000 C CNN
-F 1 "SW_Push" H 14500 2950 50  0000 C CNN
-F 2 "gamerino:B3FS-1052" H 14500 2925 50  0001 C CNN
+F 1 "HOME" H 14500 2950 50  0000 C CNN
+F 2 "gamerino:TL1220" H 14500 2925 50  0001 C CNN
 F 3 "~" H 14500 2925 50  0001 C CNN
-F 4 "B3FS-1052" H 14500 2725 50  0001 C CNN "MPN"
-F 5 "Omron" H 14500 2725 50  0001 C CNN "Manufacturer"
+F 4 "TL1220R3BBBNN" H 14500 2725 50  0001 C CNN "MPN"
+F 5 "E-Switch" H 14500 2725 50  0001 C CNN "Manufacturer"
 	1    14500 2725
 	1    0    0    -1
@@
 P 14500 3100
 F 0 "SW10" H 14500 3400 50  0000 C CNN
-F 1 "SW_Push" H 14500 3300 50  0000 C CNN
+F 1 "OPTS" H 14500 3300 50  0000 C CNN
 F 2 "gamerino:B3FS-1052" H 14500 3300 50  0001 C CNN
 F 3 "~" H 14500 3300 50  0001 C CNN
@@
 P 14500 3775
 F 0 "SW11" H 14500 4100 50  0000 C CNN
-F 1 "SW_Push" H 14500 4000 50  0000 C CNN
-F 2 "gamerino:B3FS-1052" H 14500 3975 50  0001 C CNN
+F 1 "X" H 14500 4000 50  0000 C CNN
+F 2 "gamerino:TL1220" H 14500 3975 50  0001 C CNN
 F 3 "~" H 14500 3975 50  0001 C CNN
-F 4 "B3FS-1052" H 14500 3775 50  0001 C CNN "MPN"
-F 5 "Omron" H 14500 3775 50  0001 C CNN "Manufacturer"
+F 4 "TL1220R1BBBNN" H 14500 3775 50  0001 C CNN "MPN"
+F 5 "E-Switch" H 14500 3775 50  0001 C CNN "Manufacturer"
 	1    14500 3775
 	1    0    0    -1
@@
 P 14500 4150
 F 0 "SW12" H 14500 4450 50  0000 C CNN
-F 1 "SW_Push" H 14500 4350 50  0000 C CNN
-F 2 "gamerino:B3FS-1052" H 14500 4350 50  0001 C CNN
+F 1 "B" H 14500 4350 50  0000 C CNN
+F 2 "gamerino:TL1220" H 14500 4350 50  0001 C CNN
 F 3 "~" H 14500 4350 50  0001 C CNN
-F 4 "B3FS-1052" H 14500 4150 50  0001 C CNN "MPN"
-F 5 "Omron" H 14500 4150 50  0001 C CNN "Manufacturer"
+F 4 "TL1220R1BBBNN" H 14500 4150 50  0001 C CNN "MPN"
+F 5 "E-Switch" H 14500 4150 50  0001 C CNN "Manufacturer"
 	1    14500 4150
 	1    0    0    -1
@@
 P 14500 4525
 F 0 "SW13" H 14500 4850 50  0000 C CNN
-F 1 "SW_Push" H 14500 4750 50  0000 C CNN
-F 2 "gamerino:B3FS-1052" H 14500 4725 50  0001 C CNN
+F 1 "A" H 14500 4750 50  0000 C CNN
+F 2 "gamerino:TL1220" H 14500 4725 50  0001 C CNN
 F 3 "~" H 14500 4725 50  0001 C CNN
-F 4 "B3FS-1052" H 14500 4525 50  0001 C CNN "MPN"
-F 5 "Omron" H 14500 4525 50  0001 C CNN "Manufacturer"
+F 4 "TL1220R1BBBNN" H 14500 4525 50  0001 C CNN "MPN"
+F 5 "E-Switch" H 14500 4525 50  0001 C CNN "Manufacturer"
 	1    14500 4525
 	1    0    0    -1
@@
 P 14500 4900
 F 0 "SW14" H 14500 5200 50  0000 C CNN
-F 1 "SW_Push" H 14500 5100 50  0000 C CNN
-F 2 "gamerino:B3FS-1052" H 14500 5100 50  0001 C CNN
+F 1 "Y" H 14500 5100 50  0000 C CNN
+F 2 "gamerino:TL1220" H 14500 5100 50  0001 C CNN
 F 3 "~" H 14500 5100 50  0001 C CNN
-F 4 "B3FS-1052" H 14500 4900 50  0001 C CNN "MPN"
-F 5 "Omron" H 14500 4900 50  0001 C CNN "Manufacturer"
+F 4 "TL1220R1BBBNN" H 14500 4900 50  0001 C CNN "MPN"
+F 5 "E-Switch" H 14500 4900 50  0001 C CNN "Manufacturer"
 	1    14500 4900
 	1    0    0    -1
@@
 P 14450 5600
 F 0 "SW2" H 14450 5900 50  0000 C CNN
-F 1 "SW_Push" H 14450 5800 50  0000 C CNN
-F 2 "gamerino:B3F-3155" H 14450 5800 50  0001 C CNN
+F 1 "LT1" H 14450 5800 50  0000 C CNN
+F 2 "gamerino:TL6215-R" H 14450 5800 50  0001 C CNN
 F 3 "~" H 14450 5800 50  0001 C CNN
-F 4 "B3F-3152" H 14450 5600 50  0001 C CNN "MPN"
-F 5 "Omron" H 14450 5600 50  0001 C CNN "Manufacturer"
+F 4 "TL6215RF200NDK" H 14450 5600 50  0001 C CNN "MPN"
+F 5 "E-Switch" H 14450 5600 50  0001 C CNN "Manufacturer"
 	1    14450 5600
 	-1   0    0    -1
@@
 P 14450 5975
 F 0 "SW3" H 14450 6300 50  0000 C CNN
-F 1 "SW_Push" H 14450 6200 50  0000 C CNN
-F 2 "gamerino:B3F-3155" H 14450 6175 50  0001 C CNN
+F 1 "LT2" H 14450 6200 50  0000 C CNN
+F 2 "gamerino:TL6215-R" H 14450 6175 50  0001 C CNN
 F 3 "~" H 14450 6175 50  0001 C CNN
-F 4 "B3F-3152" H 14450 5975 50  0001 C CNN "MPN"
-F 5 "Omron" H 14450 5975 50  0001 C CNN "Manufacturer"
+F 4 "TL6215RF200NDK" H 14450 5975 50  0001 C CNN "MPN"
+F 5 "E-Switch" H 14450 5975 50  0001 C CNN "Manufacturer"
 	1    14450 5975
 	-1   0    0    -1
@@
 P 14450 6350
 F 0 "SW4" H 14450 6650 50  0000 C CNN
-F 1 "SW_Push" H 14450 6550 50  0000 C CNN
-F 2 "gamerino:B3F-3155" H 14450 6550 50  0001 C CNN
+F 1 "RT1" H 14450 6550 50  0000 C CNN
+F 2 "gamerino:TL6215-R" H 14450 6550 50  0001 C CNN
 F 3 "~" H 14450 6550 50  0001 C CNN
-F 4 "B3F-3152" H 14450 6350 50  0001 C CNN "MPN"
-F 5 "Omron" H 14450 6350 50  0001 C CNN "Manufacturer"
+F 4 "TL6215RF200NDK" H 14450 6350 50  0001 C CNN "MPN"
+F 5 "E-Switch" H 14450 6350 50  0001 C CNN "Manufacturer"
 	1    14450 6350
 	-1   0    0    -1
@@
 P 14450 6725
 F 0 "SW5" H 14450 7050 50  0000 C CNN
-F 1 "SW_Push" H 14450 6950 50  0000 C CNN
-F 2 "gamerino:B3F-3155" H 14450 6925 50  0001 C CNN
+F 1 "RT2" H 14450 6950 50  0000 C CNN
+F 2 "gamerino:TL6215-R" H 14450 6925 50  0001 C CNN
 F 3 "~" H 14450 6925 50  0001 C CNN
-F 4 "B3F-3152" H 14450 6725 50  0001 C CNN "MPN"
-F 5 "Omron" H 14450 6725 50  0001 C CNN "Manufacturer"
+F 4 "TL6215RF200NDK" H 14450 6725 50  0001 C CNN "MPN"
+F 5 "E-Switch" H 14450 6725 50  0001 C CNN "Manufacturer"
 	1    14450 6725
 	-1   0    0    -1
@@
 P 14900 6925
 F 0 "#PWR036" H 14900 6675 50  0001 C CNN
-F 1 "GND" H 14925 6700 50  0000 C CNN
+F 1 "GND" H 14905 6752 50  0000 C CNN
 F 2 "" H 14900 6925 50  0001 C CNN
 F 3 "" H 14900 6925 50  0001 C CNN

Commit message: Update
Parts:
- removed D1: GREEN, LED_SMD:LED_0603_1608Metric, symbol gamerino-rescue:LED-device
- removed SW10: OPTS, gamerino:B3FS-1052, symbol gamerino-rescue:SW_Push-Switch
- removed SW11: X, gamerino:TL1220, symbol gamerino-rescue:SW_Push-Switch
- removed SW12: B, gamerino:TL1220, symbol gamerino-rescue:SW_Push-Switch
- removed SW13: A, gamerino:TL1220, symbol gamerino-rescue:SW_Push-Switch
- removed SW14: Y, gamerino:TL1220, symbol gamerino-rescue:SW_Push-Switch
- removed SW2: LT1, gamerino:TL6215-R, symbol gamerino-rescue:SW_Push-Switch
- removed SW3: LT2, gamerino:TL6215-R, symbol gamerino-rescue:SW_Push-Switch
- removed SW4: RT1, gamerino:TL6215-R, symbol gamerino-rescue:SW_Push-Switch
- removed SW5: RT2, gamerino:TL6215-R, symbol gamerino-rescue:SW_Push-Switch
- removed SW6: SEL, gamerino:B3FS-1052, symbol gamerino-rescue:SW_Push-Switch
- removed SW7: START, gamerino:B3FS-1052, symbol gamerino-rescue:SW_Push-Switch
- removed SW8: BACK, gamerino:B3FS-1052, symbol gamerino-rescue:SW_Push-Switch
- removed SW9: HOME, gamerino:TL1220, symbol gamerino-rescue:SW_Push-Switch
- added SW10: OPTS, gamerino:TL1105-T, symbol gamerino:TL1
- added SW11: X, gamerino:TL1220, symbol gamerino:TL1
- added SW12: B, gamerino:TL1220, symbol gamerino:TL1
- added SW13: A, gamerino:TL1220, symbol gamerino:TL1
- added SW14: Y, gamerino:TL1220, symbol gamerino:TL1
- added SW2: LT1, gamerino:TL6215-R, symbol gamerino:TL6
- added SW3: LT2, gamerino:TL6215-R, symbol gamerino:TL6
- added SW4: RT1, gamerino:TL6215-R, symbol gamerino:TL6
- added SW5: RT2, gamerino:TL6215-R, symbol gamerino:TL6
- added SW6: SEL, gamerino:TL1105-T, symbol gamerino:TL1
- added SW7: START, gamerino:TL1105-T, symbol gamerino:TL1
- added SW8: BACK, gamerino:TL1105-T, symbol gamerino:TL1
- added SW9: HOME, gamerino:TL1220, symbol gamerino:TL1
Connections:
- net OPTS is gone; now on net OPTIONS: U3.8 (P04)
- net +3V3: now also R4.1; no longer R4.2
- net A: now also SW13.3
- net B: now also SW12.3
- net BACK: now also SW8.3
- net GND: now also SW10.2, SW11.2, SW12.2, SW13.2, SW14.2, SW2.2, SW3.2, SW4.2, SW5.2, SW6.2, SW7.2, SW8.2, SW9.2, SW9.5
- net HOME: now also SW9.3
- net LT1: now also SW2.1
- net LT2: now also SW3.1
- net OPTIONS: now also SW10.3
- net RT1: now also SW4.1
- net RT2: now also SW5.1
- net SELECT: now also SW6.3
- net START: now also SW7.3
- net X: now also SW11.3
- net Y: now also SW14.3
- new net: R4.2, SW9.6
- no-connect marks 3 -> 21
Other:
- moved on the sheet: R4

Commit message: Update board
Parts:
- added JOY1, JOY2: RKJXU, alps:RKJXU, symbol gamerino:RKJXU
Connections:
- no-connect marks 21 -> 29
Changed lines of the file:
@@
 Wire Wire Line
 	14900 3500 14900 4325
+$Comp
+L gamerino:RKJXU JOY1
+U 1 1 60AED526
+P 10725 8075
+F 0 "JOY1" H 10650 8500 50  0000 C CNN
+F 1 "RKJXU" H 10650 8400 50  0000 C CNN
+F 2 "alps:RKJXU" H 10050 8075 50  0001 C CNN
+F 3 "" H 10050 8075 50  0001 C CNN
+F 4 "RKJXU1210006" H 10725 8075 50  0001 C CNN "MPN"
+F 5 "ALPS Alpine" H 10725 8075 50  0001 C CNN "Manufacturer"
+	1    10725 8075
+	1    0    0    -1
+$EndComp
+$Comp
+L gamerino:RKJXU JOY2
+U 1 1 60AF097E
+P 10725 6950
+F 0 "JOY2" H 10650 7400 50  0000 C CNN
+F 1 "RKJXU" H 10650 7300 50  0000 C CNN
+F 2 "alps:RKJXU" H 10050 6950 50  0001 C CNN
+F 3 "" H 10050 6950 50  0001 C CNN
+F 4 "RKJXU1210006" H 10725 6950 50  0001 C CNN "MPN"
+F 5 "ALPS Alpine" H 10725 6950 50  0001 C CNN "Manufacturer"
+	1    10725 6950
+	1    0    0    -1
+$EndComp
+NoConn ~ 10050 6950
+NoConn ~ 10050 7150
+NoConn ~ 10925 7425
+NoConn ~ 11200 6725
+NoConn ~ 11200 7850
+NoConn ~ 10050 8075
+NoConn ~ 10050 8275
+NoConn ~ 10925 8550
 $EndSCHEMATC
