File: PCB/gamerino.sch (KiCad schematic (older format))
At the start: 47 parts, among them J1 USB_B_Micro, J2 LT2, J3 RT2, P1 JOY1, P2 JOY2, P3 ICSP, P4 AUX, SW1 HATSWITCH, SW10 OPTS, SW11 X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

Commit message: Update BOM
Parts:
- C1, C2: Digikey (none) -> 478-2388-1-ND; Farnell (none) -> 1462424; Mouser (none) -> 581-TPSA106K006R1500; RS (none) -> 136-6077
- C10, C6, C7: Digikey (none) -> 732-7939-1-ND; Farnell (none) -> 2495168; Mouser (none) -> 710-885012206020; RS (none) -> 839-2720
- C3, C4: Digikey (none) -> 445-5587-1-ND; Farnell (none) -> 2210766; Mouser (none) -> 810-CGA2B2C0G1H180J; RS (none) -> 915-5538
- C5, C8, C9: Digikey (none) -> 445-12539-1-ND; Farnell (none) -> 2528789; Mouser (none) -> 810-CGA3E1X7R1C105AC; RS (none) -> 915-5660
- F1: Digikey (none) -> MF-PSMF050X-2CT-ND; Farnell (none) -> 2367280; Mouser (none) -> 652-MF-PSMF050X-2; RS (none) -> 691-7507
- J1: Digikey (none) -> A97800CT-ND; Farnell (none) -> 2751670; Mouser (none) -> 571-1981568-1; RS (none) -> 669-4645
- J2, J3: Digikey (none) -> WM1732-ND; Farnell (none) -> 9732853; Mouser (none) -> 538-53047-0310; RS (none) -> 319-1064
- JOY1, JOY2: Mouser (none) -> 688-RKJXU1210006
- P1, P2: Digikey (none) -> WM6768CT-ND; Farnell (none) -> 2679575; Mouser (none) -> 538-52746-0471; RS (none) -> 702-5438
- P3: Digikey (none) -> SAM11546-ND; Farnell (none) -> 3551038; Mouser (none) -> 200-MTLW10307GS230; RS (none) -> 208-8940
- P4: Digikey (none) -> CLM-108-02-F-D-K-TR; Farnell (none) -> 2779396; Mouser (none) -> 200-CLM10802FD; RS (none) -> 197-6486
- R1, R2: Digikey (none) -> 541-3973-1-ND; Farnell (none) -> 1469697; Mouser (none) -> 71-CRCW040222R0FKEDC; RS (none) -> 678-8983
- R3, R5, R7: Digikey (none) -> 311-10.0KHRCT-ND; Farnell (none) -> 9238603; Mouser (none) -> RC0603FR-0710KL; RS (none) -> 199-5443
- R4: Digikey (none) -> A106049CT-ND; Farnell (none) -> 3399571; Mouser (none) -> 279-CRG0603F1K0; RS (none) -> 213-2266
- R6, R8, R9: Digikey (none) -> RHM2.20KHCT-ND; Farnell (none) -> 1878615; RS (none) -> 901-3572
- SW1: Mouser (none) -> 688-RKJXS
- SW10, SW6, SW7, SW8: Digikey (none) -> EG5128CT-ND; Mouser (none) -> 612-TL6210AF200GQ
- SW11, SW12, SW13, SW14: Mouser (none) -> 612-220R1BBBNNGLOSSY
- SW9: Digikey (none) -> EG5518CT-ND; Mouser (none) -> 612-TL3265GQSCLR
- U1: Digikey (none) -> 576-1281-1-ND; Farnell (none) -> 2510252; Mouser (none) -> 998-MIC5219-3.3YM5TR; RS (none) -> 910-1685
- U2: Digikey (none) -> ATMEGA32U4-AU-ND; Farnell (none) -> 1748525; Mouser (none) -> 556-ATMEGA32U4-AU; RS (none) -> 131-0289
- X1: Digikey (none) -> 490-9650-1-ND; Farnell (none) -> 2909954; Mouser (none) -> 81-XRCHA16M000F0A1R0; RS (none) -> 144-6641

Commit message: Update BOM
Parts:
- removed U3: TCA9539, Package_SO:TSSOP-24_4.4x7.8mm_P0.65mm, symbol gamerino:TCA9539
- added U3: TCA6416A, gamerino:TSSOP-24_4.4x7.8mm_P0.65mm, symbol gamerino:TCA6416A
Changed lines of the file:
@@
-	1    0    0    -1
-$EndComp
-$Comp
-L gamerino:TCA9539 U3
-U 1 1 60A58FE8
-P 9825 4200
-F 0 "U3" H 9475 5100 50  0000 C CNN
-F 1 "TCA9539" H 10050 5100 50  0000 C CNN
-F 2 "Package_SO:TSSOP-24_4.4x7.8mm_P0.65mm" H 9425 4200 50  0001 C CNN
-F 3 "" H 9425 4200 50  0001 C CNN
-F 4 "TCA9539PWR" H 9825 4200 50  0001 C CNN "MPN"
-F 5 "TI" H 9825 4200 50  0001 C CNN "Manufacturer"
-	1    9825 4200
 	1    0    0    -1
 $EndComp
@@
 	6675 6250 7075 6250
 Wire Wire Line
-	9325 4850 9100 4850
-Wire Wire Line
-	9100 4850 9100 4950
-Wire Wire Line
 	9325 4950 9100 4950
-Connection ~ 9100 4950
 Wire Wire Line
 	9100 4950 9100 5500
@@
 U 1 1 60A6DF34
 P 8725 3550
-F 0 "R7" V 8475 3575 50  0000 C CNN
-F 1 "10K" V 8575 3575 50  0000 C CNN
+F 0 "R7" V 8517 3550 50  0000 C CNN
+F 1 "10K" V 8608 3550 50  0000 C CNN
 F 2 "Resistor_SMD:R_0603_1608Metric" V 8655 3550 30  0001 C CNN
 F 3 "" H 8725 3550 30  0000 C CNN
@@
 $EndComp
 Wire Wire Line
-	9825 3100 10025 3100
+	9825 3100 9975 3100
 Connection ~ 9825 3100
 Wire Wire Line
@@
 U 1 1 60C93238
 P 8500 4625
-F 0 "R6" H 8400 4700 50  0000 R CNN
-F 1 "2.2K" H 8400 4600 50  0000 R CNN
+F 0 "R6" H 8430 4671 50  0000 R CNN
+F 1 "2.2K" H 8430 4580 50  0000 R CNN
 F 2 "Resistor_SMD:R_0603_1608Metric" V 8430 4625 30  0001 C CNN
 F 3 "" H 8500 4625 30  0000 C CNN
@@
 U 1 1 60C9CA74
 P 8725 4625
-F 0 "R8" H 8800 4700 50  0000 L CNN
-F 1 "2.2K" H 8800 4600 50  0000 L CNN
+F 0 "R8" H 8796 4671 50  0000 L CNN
+F 1 "2.2K" H 8796 4580 50  0000 L CNN
 F 2 "Resistor_SMD:R_0603_1608Metric" V 8655 4625 30  0001 C CNN
 F 3 "" H 8725 4625 30  0000 C CNN
@@
 U 1 1 60CE92FE
 P 9225 3050
-F 0 "R9" H 9300 3100 50  0000 L CNN
-F 1 "2.2K" H 9300 3050 50  0000 L CNN
+F 0 "R9" H 9296 3096 50  0000 L CNN
+F 1 "2.2K" H 9296 3005 50  0000 L CNN
 F 2 "Resistor_SMD:R_0603_1608Metric" V 9155 3050 30  0001 C CNN
 F 3 "" H 9225 3050 30  0000 C CNN
@@
 Text Label 4725 4650 0    50   ~ 0
 D-
+$Comp
+L gamerino:TCA6416A U3
+U 1 1 60B0EB2C
+P 9825 4200
+F 0 "U3" H 10175 3075 50  0000 C CNN
+F 1 "TCA6416A" H 10200 3175 50  0000 C CNN
+F 2 "gamerino:TSSOP-24_4.4x7.8mm_P0.65mm" H 9425 4200 50  0001 C CNN
+F 3 "" H 9425 4200 50  0001 C CNN
+F 4 "TCA6416APWR" H 9825 4200 50  0001 C CNN "MPN"
+F 5 "TI" H 9825 4200 50  0001 C CNN "Manufacturer"
+F 6 "296-24536-1-ND" H 9825 4200 50  0001 C CNN "Digikey"
+F 7 "3009444" H 9825 4200 50  0001 C CNN "Farnell"
+F 8 "595-TCA6416APWR" H 9825 4200 50  0001 C CNN "Mouser"
+	1    9825 4200
+	1    0    0    -1
+$EndComp
+Wire Wire Line
+	9975 3250 9975 3100
+Connection ~ 9975 3100
+Wire Wire Line
+	9975 3100 10025 3100
 $EndSCHEMATC

Commit message: Update BOM
Parts:
- SW11, SW12, SW13, SW14: Digikey (none) -> EG6016-ND; Farnell (none) -> 2830698; MPN TL1220R1BBBNN -> TL1220R1BBBB-HALO; Mouser 612-220R1BBBNNGLOSSY -> 612-1220R1BBBRHALO
- SW2, SW3, SW4, SW5: Digikey (none) -> EG5162-ND; Farnell (none) -> TL6215RF200BDT; MPN TL6215RF200NDK -> TL6215RF200BDT; Mouser (none) -> 612-TL6215RF200BDT
Changed lines of the file:
@@
 F 2 "gamerino:TL1220" H 14475 4625 50  0001 C CNN
 F 3 "" H 14475 4625 50  0001 C CNN
-F 4 "TL1220R1BBBNN" H 14475 4475 50  0001 C CNN "MPN"
+F 4 "TL1220R1BBBB-HALO" H 14475 4475 50  0001 C CNN "MPN"
 F 5 "E-Switch" H 14475 4475 50  0001 C CNN "Manufacturer"
-F 6 "612-220R1BBBNNGLOSSY" H 14475 4475 50  0001 C CNN "Mouser"
+F 6 "612-1220R1BBBRHALO" H 14475 4475 50  0001 C CNN "Mouser"
+F 7 "EG6016-ND" H 14475 4475 50  0001 C CNN "Digikey"
+F 8 "2830698" H 14475 4475 50  0001 C CNN "Farnell"
 	1    14475 4475
 	1    0    0    -1
@@
 F 2 "gamerino:TL1220" H 14475 5725 50  0001 C CNN
 F 3 "" H 14475 5725 50  0001 C CNN
-F 4 "TL1220R1BBBNN" H 14475 5575 50  0001 C CNN "MPN"
+F 4 "TL1220R1BBBB-HALO" H 14475 5575 50  0001 C CNN "MPN"
 F 5 "E-Switch" H 14475 5575 50  0001 C CNN "Manufacturer"
-F 6 "612-220R1BBBNNGLOSSY" H 14475 5575 50  0001 C CNN "Mouser"
+F 6 "612-1220R1BBBRHALO" H 14475 5575 50  0001 C CNN "Mouser"
+F 7 "EG6016-ND" H 14475 5575 50  0001 C CNN "Digikey"
+F 8 "2830698" H 14475 5575 50  0001 C CNN "Farnell"
 	1    14475 5575
 	1    0    0    -1
@@
 F 2 "gamerino:TL1220" H 14475 6275 50  0001 C CNN
 F 3 "" H 14475 6275 50  0001 C CNN
-F 4 "TL1220R1BBBNN" H 14475 6125 50  0001 C CNN "MPN"
+F 4 "TL1220R1BBBB-HALO" H 14475 6125 50  0001 C CNN "MPN"
 F 5 "E-Switch" H 14475 6125 50  0001 C CNN "Manufacturer"
-F 6 "612-220R1BBBNNGLOSSY" H 14475 6125 50  0001 C CNN "Mouser"
+F 6 "612-1220R1BBBRHALO" H 14475 6125 50  0001 C CNN "Mouser"
+F 7 "EG6016-ND" H 14475 6125 50  0001 C CNN "Digikey"
+F 8 "2830698" H 14475 6125 50  0001 C CNN "Farnell"
 	1    14475 6125
 	1    0    0    -1
@@
 F 2 "gamerino:TL1220" H 14475 5175 50  0001 C CNN
 F 3 "" H 14475 5175 50  0001 C CNN
-F 4 "TL1220R1BBBNN" H 14475 5025 50  0001 C CNN "MPN"
+F 4 "TL1220R1BBBB-HALO" H 14475 5025 50  0001 C CNN "MPN"
 F 5 "E-Switch" H 14475 5025 50  0001 C CNN "Manufacturer"
-F 6 "612-220R1BBBNNGLOSSY" H 14475 5025 50  0001 C CNN "Mouser"
+F 6 "612-1220R1BBBRHALO" H 14475 5025 50  0001 C CNN "Mouser"
+F 7 "EG6016-ND" H 14475 5025 50  0001 C CNN "Digikey"
+F 8 "2830698" H 14475 5025 50  0001 C CNN "Farnell"
 	1    14475 5025
 	1    0    0    -1
@@
 F 2 "gamerino:TL6215-R" H 14450 6900 50  0001 C CNN
 F 3 "" H 14450 6900 50  0001 C CNN
-F 4 "TL6215RF200NDK" H 14450 6750 50  0001 C CNN "MPN"
+F 4 "TL6215RF200BDT" H 14450 6750 50  0001 C CNN "MPN"
 F 5 "E-Switch" H 14450 6750 50  0001 C CNN "Manufacturer"
+F 6 "EG5162-ND" H 14450 6750 50  0001 C CNN "Digikey"
+F 7 "TL6215RF200BDT" H 14450 6750 50  0001 C CNN "Farnell"
+F 8 "612-TL6215RF200BDT" H 14450 6750 50  0001 C CNN "Mouser"
 	1    14450 6750
 	0    -1   -1   0
@@
 F 2 "gamerino:TL6215-R" H 14450 7300 50  0001 C CNN
 F 3 "" H 14450 7300 50  0001 C CNN
-F 4 "TL6215RF200NDK" H 14450 7150 50  0001 C CNN "MPN"
+F 4 "TL6215RF200BDT" H 14450 7150 50  0001 C CNN "MPN"
 F 5 "E-Switch" H 14450 7150 50  0001 C CNN "Manufacturer"
+F 6 "EG5162-ND" H 14450 7150 50  0001 C CNN "Digikey"
+F 7 "TL6215RF200BDT" H 14450 7150 50  0001 C CNN "Farnell"
+F 8 "612-TL6215RF200BDT" H 14450 7150 50  0001 C CNN "Mouser"
 	1    14450 7150
 	0    -1   -1   0
@@
 F 2 "gamerino:TL6215-R" H 14450 7675 50  0001 C CNN
 F 3 "" H 14450 7675 50  0001 C CNN
-F 4 "TL6215RF200NDK" H 14450 7525 50  0001 C CNN "MPN"
+F 4 "TL6215RF200BDT" H 14450 7525 50  0001 C CNN "MPN"
 F 5 "E-Switch" H 14450 7525 50  0001 C CNN "Manufacturer"
+F 6 "EG5162-ND" H 14450 7525 50  0001 C CNN "Digikey"
+F 7 "TL6215RF200BDT" H 14450 7525 50  0001 C CNN "Farnell"
+F 8 "612-TL6215RF200BDT" H 14450 7525 50  0001 C CNN "Mouser"
 	1    14450 7525
 	0    -1   -1   0
@@
 F 2 "gamerino:TL6215-R" H 14450 8050 50  0001 C CNN
 F 3 "" H 14450 8050 50  0001 C CNN
-F 4 "TL6215RF200NDK" H 14450 7900 50  0001 C CNN "MPN"
+F 4 "TL6215RF200BDT" H 14450 7900 50  0001 C CNN "MPN"
 F 5 "E-Switch" H 14450 7900 50  0001 C CNN "Manufacturer"
+F 6 "EG5162-ND" H 14450 7900 50  0001 C CNN "Digikey"
+F 7 "TL6215RF200BDT" H 14450 7900 50  0001 C CNN "Farnell"
+F 8 "612-TL6215RF200BDT" H 14450 7900 50  0001 C CNN "Mouser"
 	1    14450 7900
 	0    -1   -1   0

Commit message: Update BOM
Parts:
- R6, R8, R9: Digikey RHM2.20KHCT-ND -> A129692CT-ND; Farnell 1878615 -> 2861465; MPN MCR03EZPFX2201 -> CRGCQ0603F2K2; Manufacturer ROHM -> TE; Mouser (none) -> 279-CRGCQ0603F2K2; RS 901-3572 -> 213-2317
Changed lines of the file:
@@
 F 2 "Resistor_SMD:R_0603_1608Metric" V 8430 4625 30  0001 C CNN
 F 3 "" H 8500 4625 30  0000 C CNN
-F 4 "MCR03EZPFX2201" H 8500 4625 50  0001 C CNN "MPN"
-F 5 "ROHM" H 8500 4625 50  0001 C CNN "Manufacturer"
-F 6 "RHM2.20KHCT-ND" H 8500 4625 50  0001 C CNN "Digikey"
-F 7 "901-3572" H 8500 4625 50  0001 C CNN "RS"
-F 8 "1878615" H 8500 4625 50  0001 C CNN "Farnell"
+F 4 "CRGCQ0603F2K2" H 8500 4625 50  0001 C CNN "MPN"
+F 5 "TE" H 8500 4625 50  0001 C CNN "Manufacturer"
+F 6 "A129692CT-ND" H 8500 4625 50  0001 C CNN "Digikey"
+F 7 "213-2317" H 8500 4625 50  0001 C CNN "RS"
+F 8 "2861465" H 8500 4625 50  0001 C CNN "Farnell"
+F 9 "279-CRGCQ0603F2K2" H 8500 4625 50  0001 C CNN "Mouser"
 	1    8500 4625
 	1    0    0    -1
@@
 F 2 "Resistor_SMD:R_0603_1608Metric" V 8655 4625 30  0001 C CNN
 F 3 "" H 8725 4625 30  0000 C CNN
-F 4 "MCR03EZPFX2201" H 8725 4625 50  0001 C CNN "MPN"
-F 5 "ROHM" H 8725 4625 50  0001 C CNN "Manufacturer"
-F 6 "RHM2.20KHCT-ND" H 8725 4625 50  0001 C CNN "Digikey"
-F 7 "901-3572" H 8725 4625 50  0001 C CNN "RS"
-F 8 "1878615" H 8725 4625 50  0001 C CNN "Farnell"
+F 4 "CRGCQ0603F2K2" H 8725 4625 50  0001 C CNN "MPN"
+F 5 "TE" H 8725 4625 50  0001 C CNN "Manufacturer"
+F 6 "A129692CT-ND" H 8725 4625 50  0001 C CNN "Digikey"
+F 7 "213-2317" H 8725 4625 50  0001 C CNN "RS"
+F 8 "2861465" H 8725 4625 50  0001 C CNN "Farnell"
+F 9 "279-CRGCQ0603F2K2" H 8725 4625 50  0001 C CNN "Mouser"
 	1    8725 4625
 	1    0    0    -1
@@
 F 2 "Resistor_SMD:R_0603_1608Metric" V 9155 3050 30  0001 C CNN
 F 3 "" H 9225 3050 30  0000 C CNN
-F 4 "MCR03EZPFX2201" H 9225 3050 50  0001 C CNN "MPN"
-F 5 "ROHM" H 9225 3050 50  0001 C CNN "Manufacturer"
-F 6 "RHM2.20KHCT-ND" H 9225 3050 50  0001 C CNN "Digikey"
-F 7 "901-3572" H 9225 3050 50  0001 C CNN "RS"
-F 8 "1878615" H 9225 3050 50  0001 C CNN "Farnell"
+F 4 "CRGCQ0603F2K2" H 9225 3050 50  0001 C CNN "MPN"
+F 5 "TE" H 9225 3050 50  0001 C CNN "Manufacturer"
+F 6 "A129692CT-ND" H 9225 3050 50  0001 C CNN "Digikey"
+F 7 "213-2317" H 9225 3050 50  0001 C CNN "RS"
+F 8 "2861465" H 9225 3050 50  0001 C CNN "Farnell"
+F 9 "279-CRGCQ0603F2K2" H 9225 3050 50  0001 C CNN "Mouser"
 	1    9225 3050
 	1    0    0    -1

Commit message: Update BOM
Parts:
- SW2, SW3, SW4, SW5: Farnell TL6215RF200BDT -> 2830788
Changed lines of the file:
@@
 F 5 "E-Switch" H 14450 6750 50  0001 C CNN "Manufacturer"
 F 6 "EG5162-ND" H 14450 6750 50  0001 C CNN "Digikey"
-F 7 "TL6215RF200BDT" H 14450 6750 50  0001 C CNN "Farnell"
+F 7 "2830788" H 14450 6750 50  0001 C CNN "Farnell"
 F 8 "612-TL6215RF200BDT" H 14450 6750 50  0001 C CNN "Mouser"
 	1    14450 6750
@@
 F 5 "E-Switch" H 14450 7150 50  0001 C CNN "Manufacturer"
 F 6 "EG5162-ND" H 14450 7150 50  0001 C CNN "Digikey"
-F 7 "TL6215RF200BDT" H 14450 7150 50  0001 C CNN "Farnell"
+F 7 "2830788" H 14450 7150 50  0001 C CNN "Farnell"
 F 8 "612-TL6215RF200BDT" H 14450 7150 50  0001 C CNN "Mouser"
 	1    14450 7150
@@
 F 5 "E-Switch" H 14450 7525 50  0001 C CNN "Manufacturer"
 F 6 "EG5162-ND" H 14450 7525 50  0001 C CNN "Digikey"
-F 7 "TL6215RF200BDT" H 14450 7525 50  0001 C CNN "Farnell"
+F 7 "2830788" H 14450 7525 50  0001 C CNN "Farnell"
 F 8 "612-TL6215RF200BDT" H 14450 7525 50  0001 C CNN "Mouser"
 	1    14450 7525
@@
 F 5 "E-Switch" H 14450 7900 50  0001 C CNN "Manufacturer"
 F 6 "EG5162-ND" H 14450 7900 50  0001 C CNN "Digikey"
-F 7 "TL6215RF200BDT" H 14450 7900 50  0001 C CNN "Farnell"
+F 7 "2830788" H 14450 7900 50  0001 C CNN "Farnell"
 F 8 "612-TL6215RF200BDT" H 14450 7900 50  0001 C CNN "Mouser"
 	1    14450 7900

Commit message: Routing
Parts:
- SW8: value BACK -> CLEAR
Connections:
- net BACK is gone; now on net CLEAR: SW8.3
- net IRQ: now also U2.12 (PB7); no longer U2.8 (PB0)
- net PB4: now also P4.7; no longer P4.14
- net PB5: now also P4.5; no longer P4.12
- net PC7: now also P4.3; no longer P4.2
- net PD3: now also P4.12; no longer P4.13
- net PD4: now also P4.13; no longer P4.11
- net PD5: now also P4.14; no longer P4.9
- net PD6: now also P4.11; no longer P4.7
- net PD7: now also P4.9; no longer P4.5
- net PE6: now also P4.2; no longer P4.3
- net XTAL1: now also X1.1; no longer X1.2
- net XTAL2: now also X1.2; no longer X1.1
- net PB7 renamed PB0
- net PB0: now also U2.8 (PB0); no longer U2.12 (PB7)
Changed lines of the file:
@@
 U 1 1 60A7134E
 P 4325 6125
-F 0 "X1" V 4400 5950 50  0000 R CNN
-F 1 "16MHz" V 4300 5950 50  0000 R CNN
+F 0 "X1" V 4279 6258 50  0000 L CNN
+F 1 "16MHz" V 4370 6258 50  0000 L CNN
 F 2 "Crystal:Crystal_SMD_2520-4Pin_2.5x2.0mm" H 4325 6125 60  0001 C CNN
 F 3 "" H 4325 6125 60  0001 C CNN
@@
 F 9 "2909954" H 4325 6125 50  0001 C CNN "Farnell"
 	1    4325 6125
-	0    -1   -1   0
+	0    1    1    0
 $EndComp
 $Comp
@@
 $EndComp
 Wire Wire Line
-	4175 5825 4325 5825
-Connection ~ 4325 5825
-Wire Wire Line
-	4175 6425 4325 6425
-Connection ~ 4325 6425
-Wire Wire Line
 	3775 5825 3625 5825
 Wire Wire Line
@@
 Wire Wire Line
 	5475 3950 4975 3950
-Wire Wire Line
-	4325 5825 4800 5825
-Wire Wire Line
-	4325 6425 4800 6425
 Wire Wire Line
 	6675 6350 7075 6350
@@
 SDA
 Text Label 9100 3450 2    50   ~ 0
-IRQ
-Text Label 7075 3550 0    50   ~ 0
 IRQ
 Wire Wire Line
@@
 Text Label 13900 2125 2    50   ~ 0
 START
-Text Label 13900 2675 2    50   ~ 0
-BACK
 Text Label 13900 3800 2    50   ~ 0
 OPTIONS
@@
 Wire Wire Line
 	6475 8175 6875 8175
+Text Label 6875 8075 0    50   ~ 0
+PD4
+Wire Wire Line
+	6475 8275 6875 8275
+Text Label 5275 8075 2    50   ~ 0
+PD5
+Wire Wire Line
+	6475 8375 6875 8375
 Text Label 6875 8175 0    50   ~ 0
-PD4
-Wire Wire Line
-	6475 8275 6875 8275
+PD6
+Wire Wire Line
+	6475 8475 6875 8475
 Text Label 6875 8275 0    50   ~ 0
-PD5
-Wire Wire Line
-	6475 8375 6875 8375
-Text Label 6875 8375 0    50   ~ 0
-PD6
-Wire Wire Line
-	6475 8475 6875 8475
-Text Label 6875 8475 0    50   ~ 0
 PD7
 Wire Wire Line
@@
 Wire Wire Line
 	6475 8075 6875 8075
-Text Label 6875 8075 0    50   ~ 0
+Text Label 5275 8175 2    50   ~ 0
 PD3
-Text Label 7075 4250 0    50   ~ 0
-PB7
 Wire Wire Line
 	6675 4250 7075 4250
@@
 	6675 3850 7075 3850
 Text Label 5275 8375 2    50   ~ 0
-PB7
+PB0
 Wire Wire Line
 	5675 8375 5275 8375
@@
 Wire Wire Line
 	5675 8275 5275 8275
-Text Label 5275 8175 2    50   ~ 0
+Text Label 6875 8475 0    50   ~ 0
 PB5
 Wire Wire Line
 	5675 8175 5275 8175
-Text Label 5275 8075 2    50   ~ 0
+Text Label 6875 8375 0    50   ~ 0
 PB4
 Wire Wire Line
@@
 Wire Wire Line
 	5675 8675 5275 8675
-Text Label 5275 8675 2    50   ~ 0
+Text Label 6875 8575 0    50   ~ 0
 PC7
 NoConn ~ 5675 8475
 Wire Wire Line
 	6475 8575 6875 8575
-Text Label 6875 8575 0    50   ~ 0
+Text Label 5275 8675 2    50   ~ 0
 PE6
 $Comp
@@
 P 14450 2525
 F 0 "SW8" H 14467 2856 50  0000 C CNN
-F 1 "BACK" H 14467 2765 50  0000 C CNN
+F 1 "CLEAR" H 14467 2765 50  0000 C CNN
 F 2 "gamerino:TL6210" H 14450 2175 50  0001 C CNN
 F 3 "" H 14450 2175 50  0001 C CNN
@@
 Wire Wire Line
 	9975 3100 10025 3100
+Wire Wire Line
+	4175 5825 4325 5825
+Wire Wire Line
+	4175 6425 4325 6425
+Connection ~ 4325 5825
+Wire Wire Line
+	4325 5825 4800 5825
+Connection ~ 4325 6425
+Wire Wire Line
+	4325 6425 4800 6425
+Text Label 13900 2675 2    50   ~ 0
+CLEAR
+Text Label 7075 4250 0    50   ~ 0
+IRQ
+Text Label 7075 3550 0    50   ~ 0
+PB0
 $EndSCHEMATC
