File: PCB/gamerino.sch (KiCad schematic (older format))
At the start: 51 parts, among them J1 USB_B_Micro, J2 LT2, J3 RT2, P1 JOY1, P2 JOY2, P3 ICSP, P4 AUX, SW1 HATSWITCH, SW10 OPTS, SW11 X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

Commit message: Update
Parts:
- added D5, D6: NSR0520V2T1G, Diode_SMD:D_SOD-523, symbol Device:D
- added J4: ACT1, gamerino:Molex_PicoBlade_53047-0210_1x02_P1.25mm_Vertical, symbol Connector:Conn_01x02_Male
- added J5: ACT2, gamerino:Molex_PicoBlade_53047-0210_1x02_P1.25mm_Vertical, symbol Connector:Conn_01x02_Male
- added Q1, Q2: DMN601WK, Package_TO_SOT_SMD:SOT-323_SC-70, symbol Device:Q_NMOS_GSD
- added R10, R12: 0R, Resistor_SMD:R_0603_1608Metric, symbol gamerino-rescue:R-device
- added R11, R13: 10K, Resistor_SMD:R_0603_1608Metric, symbol gamerino-rescue:R-device
Connections:
- net +3V3: now also D5.1 (K), D6.1 (K), J4.2 (Pin_2), J5.2 (Pin_2)
- net GND: now also Q1.2 (S), Q2.2 (S), R11.1, R13.1
- net PD2: now also R10.2
- net PD3: now also R12.2
- new net: Q2.1 (G), R12.1, R13.2
- new net: Q1.1 (G), R10.1, R11.2
- new net ACT1-: D5.2 (A), J4.1 (Pin_1), Q1.3 (D)
- new net ACT2-: D6.2 (A), J5.1 (Pin_1), Q2.3 (D)

Commit message: Update docs, layout optimization, teardrops
Parts:
- J2, J3: symbol gamerino-rescue:CONN_3-conn -> Connector:Conn_01x03_Male
- P1, P2: symbol gamerino-rescue:CONN_4-conn -> Connector:Conn_01x04_Male
Connections:
- net PE6 is gone; now on net IRQ: U2.1 (PE6)
- net IRQ: no longer U2.12 (PB7)
- new net PB7: U2.12 (PB7)
Changed lines of the file:
@@
 	6675 6250 7075 6250
 $Comp
-L gamerino-rescue:CONN_4-conn P1
+L Connector:Conn_01x04_Male P1
 U 1 1 60A872FE
-P 4225 8125
-F 0 "P1" H 4100 7700 50  0000 C CNN
-F 1 "JOY1" H 4100 7800 50  0000 C CNN
-F 2 "gamerino:52746-0471" H 4225 8125 50  0001 C CNN
-F 3 "" H 4225 8125 50  0001 C CNN
-F 4 "52746-0471" H 4225 8125 50  0001 C CNN "MPN"
-F 5 "Molex" H 4225 8125 50  0001 C CNN "Manufacturer"
-F 6 "WM6768CT-ND" H 4225 8125 50  0001 C CNN "Digikey"
-F 7 "538-52746-0471" H 4225 8125 50  0001 C CNN "Mouser"
-F 8 "702-5438" H 4225 8125 50  0001 C CNN "RS"
-F 9 "2679575" H 4225 8125 50  0001 C CNN "Farnell"
-	1    4225 8125
-	1    0    0    1
-$EndComp
-$Comp
-L gamerino-rescue:CONN_4-conn P2
+P 4075 8175
+F 0 "P1" H 3950 7750 50  0000 C CNN
+F 1 "JOY1" H 3950 7850 50  0000 C CNN
+F 2 "gamerino:52746-0471" H 4075 8175 50  0001 C CNN
+F 3 "" H 4075 8175 50  0001 C CNN
+F 4 "52746-0471" H 4075 8175 50  0001 C CNN "MPN"
+F 5 "Molex" H 4075 8175 50  0001 C CNN "Manufacturer"
+F 6 "WM6768CT-ND" H 4075 8175 50  0001 C CNN "Digikey"
+F 7 "538-52746-0471" H 4075 8175 50  0001 C CNN "Mouser"
+F 8 "702-5438" H 4075 8175 50  0001 C CNN "RS"
+F 9 "2679575" H 4075 8175 50  0001 C CNN "Farnell"
+	1    4075 8175
+	-1   0    0    1
+$EndComp
+$Comp
+L Connector:Conn_01x04_Male P2
 U 1 1 60A87A63
-P 4225 8700
-F 0 "P2" H 4400 8600 50  0000 L CNN
-F 1 "JOY2" H 4400 8700 50  0000 L CNN
-F 2 "gamerino:52746-0471" H 4225 8700 50  0001 C CNN
-F 3 "" H 4225 8700 50  0001 C CNN
-F 4 "52746-0471" H 4225 8700 50  0001 C CNN "MPN"
-F 5 "Molex" H 4225 8700 50  0001 C CNN "Manufacturer"
-F 6 "WM6768CT-ND" H 4225 8700 50  0001 C CNN "Digikey"
-F 7 "538-52746-0471" H 4225 8700 50  0001 C CNN "Mouser"
-F 8 "702-5438" H 4225 8700 50  0001 C CNN "RS"
-F 9 "2679575" H 4225 8700 50  0001 C CNN "Farnell"
-	1    4225 8700
-	1    0    0    1
+P 4075 8750
+F 0 "P2" H 4047 8632 50  0000 R CNN
+F 1 "JOY2" H 4047 8723 50  0000 R CNN
+F 2 "gamerino:52746-0471" H 4075 8750 50  0001 C CNN
+F 3 "" H 4075 8750 50  0001 C CNN
+F 4 "52746-0471" H 4075 8750 50  0001 C CNN "MPN"
+F 5 "Molex" H 4075 8750 50  0001 C CNN "Manufacturer"
+F 6 "WM6768CT-ND" H 4075 8750 50  0001 C CNN "Digikey"
+F 7 "538-52746-0471" H 4075 8750 50  0001 C CNN "Mouser"
+F 8 "702-5438" H 4075 8750 50  0001 C CNN "RS"
+F 9 "2679575" H 4075 8750 50  0001 C CNN "Farnell"
+	1    4075 8750
+	-1   0    0    1
 $EndComp
 Wire Wire Line
@@
 PC7
 Wire Wire Line
-	6675 5750 7075 5750
-Text Label 7075 5750 0    50   ~ 0
-PE6
+	6675 4250 7075 4250
+Text Label 7075 4250 0    50   ~ 0
+PB7
 Wire Wire Line
 	7675 5650 7950 5650
@@
 	5900 8175 6300 8175
 Wire Wire Line
-	6675 4250 7075 4250
+	6675 5750 7075 5750
 Text Label 7075 4150 0    50   ~ 0
 PB6
@@
 	5900 8775 6300 8775
 $Comp
-L gamerino-rescue:CONN_3-conn J3
+L Connector:Conn_01x03_Male J3
 U 1 1 61121A56
-P 8175 9925
-F 0 "J3" H 8050 9550 50  0000 C CNN
-F 1 "RT2" H 8050 9650 50  0000 C CNN
-F 2 "gamerino:Molex_PicoBlade_53047-0310_1x03_P1.25mm_Vertical" H 8175 9925 50  0001 C CNN
-F 3 "" H 8175 9925 50  0001 C CNN
-F 4 "53047-0310" H 8175 9925 50  0001 C CNN "MPN"
-F 5 "Molex" H 8175 9925 50  0001 C CNN "Manufacturer"
-F 6 "WM1732-ND" H 8175 9925 50  0001 C CNN "Digikey"
-F 7 "538-53047-0310" H 8175 9925 50  0001 C CNN "Mouser"
-F 8 "319-1064" H 8175 9925 50  0001 C CNN "RS"
-F 9 "9732853" H 8175 9925 50  0001 C CNN "Farnell"
-	1    8175 9925
-	1    0    0    1
+P 8025 9925
+F 0 "J3" H 7997 9857 50  0000 R CNN
+F 1 "RT2" H 7997 9948 50  0000 R CNN
+F 2 "gamerino:Molex_PicoBlade_53047-0310_1x03_P1.25mm_Vertical" H 8025 9925 50  0001 C CNN
+F 3 "" H 8025 9925 50  0001 C CNN
+F 4 "53047-0310" H 8025 9925 50  0001 C CNN "MPN"
+F 5 "Molex" H 8025 9925 50  0001 C CNN "Manufacturer"
+F 6 "WM1732-ND" H 8025 9925 50  0001 C CNN "Digikey"
+F 7 "538-53047-0310" H 8025 9925 50  0001 C CNN "Mouser"
+F 8 "319-1064" H 8025 9925 50  0001 C CNN "RS"
+F 9 "9732853" H 8025 9925 50  0001 C CNN "Farnell"
+	1    8025 9925
+	-1   0    0    1
 $EndComp
 $Comp
@@
 	7825 8275 7825 8600
 $Comp
-L gamerino-rescue:CONN_3-conn J2
+L Connector:Conn_01x03_Male J2
 U 1 1 6116B2CB
-P 8175 8175
-F 0 "J2" H 8042 7839 50  0000 C CNN
-F 1 "LT2" H 8042 7930 50  0000 C CNN
-F 2 "gamerino:Molex_PicoBlade_53047-0310_1x03_P1.25mm_Vertical" H 8175 8175 50  0001 C CNN
-F 3 "" H 8175 8175 50  0001 C CNN
-F 4 "53047-0310" H 8175 8175 50  0001 C CNN "MPN"
-F 5 "Molex" H 8175 8175 50  0001 C CNN "Manufacturer"
-F 6 "WM1732-ND" H 8175 8175 50  0001 C CNN "Digikey"
-F 7 "538-53047-0310" H 8175 8175 50  0001 C CNN "Mouser"
-F 8 "319-1064" H 8175 8175 50  0001 C CNN "RS"
-F 9 "9732853" H 8175 8175 50  0001 C CNN "Farnell"
-	1    8175 8175
-	1    0    0    1
+P 8025 8175
+F 0 "J2" H 7997 8107 50  0000 R CNN
+F 1 "LT2" H 7997 8198 50  0000 R CNN
+F 2 "gamerino:Molex_PicoBlade_53047-0310_1x03_P1.25mm_Vertical" H 8025 8175 50  0001 C CNN
+F 3 "" H 8025 8175 50  0001 C CNN
+F 4 "53047-0310" H 8025 8175 50  0001 C CNN "MPN"
+F 5 "Molex" H 8025 8175 50  0001 C CNN "Manufacturer"
+F 6 "WM1732-ND" H 8025 8175 50  0001 C CNN "Digikey"
+F 7 "538-53047-0310" H 8025 8175 50  0001 C CNN "Mouser"
+F 8 "319-1064" H 8025 8175 50  0001 C CNN "RS"
+F 9 "9732853" H 8025 8175 50  0001 C CNN "Farnell"
+	1    8025 8175
+	-1   0    0    1
 $EndComp
 $Comp
@@
 Text Label 15000 2375 0    50   ~ 0
 CLEAR
-Text Label 7075 4250 0    50   ~ 0
+Text Label 7075 5750 0    50   ~ 0
 IRQ
 Text Label 7075 3550 0    50   ~ 0

Commit message: Update
Parts:
- P4: Digikey 2073-BC070-10-A-1-L-CCT-ND -> 952-1844-ND; Farnell (none) -> 1099544; MPN BC070-10-A-1-L-C -> M52-50010045; Manufacturer GCT -> Harwin; Mouser 640-BC070-10-A-1-L-C -> 855-M52-5001045; RS (none) -> 681-3032
Changed lines of the file:
@@
 F 2 "Connector_PinSocket_1.00mm:PinSocket_1x10_P1.00mm_Vertical_SMD_Pin1Left" H 5700 8475 50  0001 C CNN
 F 3 "" H 5700 8475 50  0001 C CNN
-F 4 "2073-BC070-10-A-1-L-CCT-ND" H 5700 8475 50  0001 C CNN "Digikey"
-F 5 "BC070-10-A-1-L-C" H 5700 8475 50  0001 C CNN "MPN"
-F 6 "GCT" H 5700 8475 50  0001 C CNN "Manufacturer"
-F 7 "640-BC070-10-A-1-L-C" H 5700 8475 50  0001 C CNN "Mouser"
+F 4 "952-1844-ND" H 5700 8475 50  0001 C CNN "Digikey"
+F 5 "M52-50010045" H 5700 8475 50  0001 C CNN "MPN"
+F 6 "Harwin" H 5700 8475 50  0001 C CNN "Manufacturer"
+F 7 "855-M52-5001045" H 5700 8475 50  0001 C CNN "Mouser"
+F 8 "1099544" H 5700 8475 50  0001 C CNN "Farnell"
+F 9 "681-3032" H 5700 8475 50  0001 C CNN "RS"
 	1    5700 8475
 	-1   0    0    1

Commit message: Update
Parts:
- added D7: ESDS304, Package_TO_SOT_SMD:SOT-23-5, symbol gamerino:ESDS304
Connections:
- net D+: now also D7.5 (K4)
- net D-: now also D7.4 (K3)
- net GND: now also D7.2 (A)
- net VBUS: now also D7.3 (K2)
- no-connect marks 28 -> 29
Changed lines of the file:
@@
 	1    0    0    -1
 $EndComp
+$Comp
+L gamerino:ESDS304 D7
+U 1 1 60C3C328
+P 10400 1700
+F 0 "D7" V 10354 1768 50  0000 L CNN
+F 1 "ESDS304" V 10445 1768 50  0000 L CNN
+F 2 "Package_TO_SOT_SMD:SOT-23-5" H 10400 1700 50  0001 C CNN
+F 3 "" H 10400 1700 50  0001 C CNN
+F 4 "296-ESDS304DBVRCT-ND" H 10400 1700 50  0001 C CNN "Digikey"
+F 5 "ESDS304DBVR" H 10400 1700 50  0001 C CNN "MPN"
+F 6 "TI" H 10400 1700 50  0001 C CNN "Manufacturer"
+F 7 "595-ESDS304DBVR" H 10400 1700 50  0001 C CNN "Mouser"
+	1    10400 1700
+	0    1    1    0
+$EndComp
+$Comp
+L gamerino:ESDS304 D7
+U 2 1 60C53CCB
+P 9825 1700
+F 0 "D7" V 9741 1768 50  0000 L CNN
+F 1 "ESDS304" V 9832 1768 50  0000 L CNN
+F 2 "Package_TO_SOT_SMD:SOT-23-5" H 9825 1700 50  0001 C CNN
+F 3 "" H 9825 1700 50  0001 C CNN
+F 4 "296-ESDS304DBVRCT-ND" H 9825 1700 50  0001 C CNN "Digikey"
+F 5 "ESDS304DBVR" H 9825 1700 50  0001 C CNN "MPN"
+F 6 "TI" H 9825 1700 50  0001 C CNN "Manufacturer"
+F 7 "595-ESDS304DBVR" H 9825 1700 50  0001 C CNN "Mouser"
+	2    9825 1700
+	0    1    1    0
+$EndComp
+$Comp
+L gamerino:ESDS304 D7
+U 3 1 60C55212
+P 9225 1700
+F 0 "D7" V 9141 1768 50  0000 L CNN
+F 1 "ESDS304" V 9232 1768 50  0000 L CNN
+F 2 "Package_TO_SOT_SMD:SOT-23-5" H 9225 1700 50  0001 C CNN
+F 3 "" H 9225 1700 50  0001 C CNN
+F 4 "296-ESDS304DBVRCT-ND" H 9225 1700 50  0001 C CNN "Digikey"
+F 5 "ESDS304DBVR" H 9225 1700 50  0001 C CNN "MPN"
+F 6 "TI" H 9225 1700 50  0001 C CNN "Manufacturer"
+F 7 "595-ESDS304DBVR" H 9225 1700 50  0001 C CNN "Mouser"
+	3    9225 1700
+	0    1    1    0
+$EndComp
+Wire Wire Line
+	10400 1800 10400 1925
+$Comp
+L gamerino-rescue:GND-power #PWR0113
+U 1 1 60C6DE4E
+P 10400 1925
+F 0 "#PWR0113" H 10400 1675 50  0001 C CNN
+F 1 "GND" H 10405 1752 50  0000 C CNN
+F 2 "" H 10400 1925 50  0001 C CNN
+F 3 "" H 10400 1925 50  0001 C CNN
+	1    10400 1925
+	1    0    0    -1
+$EndComp
+Text Label 8625 1450 0    50   ~ 0
+D+
+Text Label 9225 1450 0    50   ~ 0
+D-
+$Comp
+L gamerino-rescue:VBUS-power #PWR0114
+U 1 1 60C6E35D
+P 9825 1450
+F 0 "#PWR0114" H 9825 1300 50  0001 C CNN
+F 1 "VBUS" H 9950 1525 50  0000 L CNN
+F 2 "" H 9825 1450 50  0001 C CNN
+F 3 "" H 9825 1450 50  0001 C CNN
+	1    9825 1450
+	1    0    0    -1
+$EndComp
+Wire Wire Line
+	9825 1600 9825 1450
+Wire Wire Line
+	9225 1600 9225 1450
+Wire Wire Line
+	8625 1600 8625 1450
+$Comp
+L gamerino:ESDS304 D7
+U 4 1 60D53CF1
+P 8625 1700
+F 0 "D7" V 8541 1768 50  0000 L CNN
+F 1 "ESDS304" V 8632 1768 50  0000 L CNN
+F 2 "Package_TO_SOT_SMD:SOT-23-5" H 8625 1700 50  0001 C CNN
+F 3 "" H 8625 1700 50  0001 C CNN
+F 4 "296-ESDS304DBVRCT-ND" H 8625 1700 50  0001 C CNN "Digikey"
+F 5 "ESDS304DBVR" H 8625 1700 50  0001 C CNN "MPN"
+F 6 "TI" H 8625 1700 50  0001 C CNN "Manufacturer"
+F 7 "595-ESDS304DBVR" H 8625 1700 50  0001 C CNN "Mouser"
+	4    8625 1700
+	0    1    1    0
+$EndComp
+NoConn ~ 10400 1600
 $EndSCHEMATC

Commit message: Update
Parts:
- SW9: Digikey EG5518CT-ND -> EG5517CT-ND; MPN TL3265GQSCLR -> TL3265BQSCLR; Mouser 612-TL3265GQSCLR -> 612-TL3265BQSCLR
Changed lines of the file:
@@
 F 2 "gamerino:TL3265" H 14450 3250 50  0001 C CNN
 F 3 "" H 14450 3250 50  0001 C CNN
-F 4 "TL3265GQSCLR" H 14450 3100 50  0001 C CNN "MPN"
+F 4 "TL3265BQSCLR" H 14450 3100 50  0001 C CNN "MPN"
 F 5 "E-Switch" H 14450 3100 50  0001 C CNN "Manufacturer"
-F 6 "EG5518CT-ND" H 14450 3100 50  0001 C CNN "Digikey"
-F 7 "612-TL3265GQSCLR" H 14450 3100 50  0001 C CNN "Mouser"
+F 6 "EG5517CT-ND" H 14450 3100 50  0001 C CNN "Digikey"
+F 7 "612-TL3265BQSCLR" H 14450 3100 50  0001 C CNN "Mouser"
 	1    14450 3100
 	1    0    0    -1
@@
 F 2 "gamerino:TL3265" H 8800 8325 50  0001 C CNN
 F 3 "" H 8800 8325 50  0001 C CNN
-F 4 "TL3265GQSCLR" H 8800 8175 50  0001 C CNN "MPN"
+F 4 "TL3265BQSCLR" H 8800 8175 50  0001 C CNN "MPN"
 F 5 "E-Switch" H 8800 8175 50  0001 C CNN "Manufacturer"
-F 6 "EG5518CT-ND" H 8800 8175 50  0001 C CNN "Digikey"
-F 7 "612-TL3265GQSCLR" H 8800 8175 50  0001 C CNN "Mouser"
+F 6 "EG5517CT-ND" H 8800 8175 50  0001 C CNN "Digikey"
+F 7 "612-TL3265BQSCLR" H 8800 8175 50  0001 C CNN "Mouser"
 	2    8800 8175
 	0    -1   -1   0
