File: PCB/gamerino.kicad_pcb (KiCad board)
At the start: 2 copper layers, 91.4 x 63.5 mm, 46 parts, among them J1 USB_B_Micro, J2 LT2, J3 RT2, P1 JOY1, P2 JOY2, P3 ICSP, P4 AUX, SW1 HATSWITCH, SW10 SW_Push, SW11 SW_Push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

Commit message: Update
Parts:
- J2, J3: footprint Connector_Molex:Molex_PicoBlade_53047-0310_1x03_P1.25mm_Vertical -> gamerino:53398-0371
- R6, R7, R8, R9, SW3, SW5: moved to B.Cu
- SW10, SW11, SW12, SW13, SW14, SW6, SW7, SW8, SW9: footprint gamerino:B3FS-1052 -> gamerino:B3W-1050
- SW2, SW4: moved to F.Cu
- moved SW5 113.4 mm to (170.4, 59.5), turned to 0 degrees
- moved SW4 113.3 mm to (180.5, 59.5), turned to 180 degrees
- moved C2 106.1 mm to (151.5, 64.0), turned to 180 degrees
- moved C1 95.6 mm to (144.0, 65.0), turned to 270 degrees
- moved F1 89.1 mm to (144.0, 69.0), turned to 90 degrees
- moved D1 84.7 mm to (151.0, 78.5), turned to 90 degrees
- moved C6 64.0 mm to (150.5, 67.5)
- moved P2 61.5 mm to (100.5, 112.5), turned to 180 degrees
- moved SW11 59.4 mm to (191.5, 78.0)
- moved U1 56.8 mm to (147.0, 65.0)
- moved SW7 56.1 mm to (180.5, 89.0)
- moved C5 54.2 mm to (150.5, 66.0)
- moved C9 54.0 mm to (141.5, 85.0), turned to 90 degrees
- moved SW13 54.0 mm to (180.5, 67.0)
- moved R9 53.2 mm to (144.0, 85.0), turned to 270 degrees
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Routing:
- net Net-(R2-Pad1): track 0.00 -> 20.8 mm
- net Net-(R1-Pad1): track 0.00 -> 20.3 mm
- net Net-(J1-Pad3): track 0.00 -> 2.77 mm
- net Net-(J1-Pad2): track 0.00 -> 2.75 mm
- added copper zone on F.Cu, net GND
Other:
- board size 91.4 x 63.5 mm -> 125 x 60 mm

Commit message: Update
Parts:
- removed D1: GREEN, LED_SMD:LED_0603_1608Metric
- R4: moved to B.Cu
- SW11, SW13, SW7, SW8, SW9: footprint gamerino:B3W-1050 -> gamerino:TL1220
- SW2, SW3, SW4, SW5: footprint gamerino:B3F-3155 -> gamerino:TL6215-R
- moved R4 13.1 mm to (138.0, 76.5)
- moved SW10 3.00 mm to (160.5, 60.0)
- moved SW12 3.00 mm to (115.5, 60.0)
- moved SW3 1.12 mm to (106.5, 59.0)
- moved SW5 1.05 mm to (169.5, 59.0)
- moved J2 1.00 mm to (169.5, 68.5)
- moved J3 1.00 mm to (106.5, 68.5)
- moved SW2 0.50 mm to (95.5, 59.0)
- moved SW4 0.50 mm to (180.5, 59.0)
Routing:
- net Net-(R2-Pad1): track 20.8 -> 0.00 mm
- net Net-(R1-Pad1): track 20.3 -> 0.00 mm
Other:
- board size 125 x 60 mm -> 125 x 63 mm

Commit message: Update
Parts:
- removed the SW13 at (180.5, 67.0)
- added SW14: Y, gamerino:TL1220, F.Cu at (180.5, 67.0)
- added h1: MountingHole_2mm, MountingHole:MountingHole_2mm, F.Cu at (103.1, 68.3)
- added h2: MountingHole_1.5mm, gamerino:MountingHole_1.5mm, F.Cu at (88.0, 69.6)
- added h3: MountingHole_1.5mm, gamerino:MountingHole_1.5mm, F.Cu at (168.1, 111.4)
- added h4: MountingHole_2mm, MountingHole:MountingHole_2mm, F.Cu at (152.9, 112.7)
- J2: footprint gamerino:53398-0371 -> Connector_Molex:Molex_PicoBlade_53047-0310_1x03_P1.25mm_Vertical
- J3: footprint gamerino:53398-0371 -> gamerino:Molex_PicoBlade_53047-0310_1x03_P1.25mm_Vertical
- SW10: renamed from SW14; value SW_Push -> OPTS; footprint gamerino:B3W-1050 -> gamerino:TL1105-T
- SW11: renamed from SW8; value SW_Push -> X
- SW12: renamed from SW11; value SW_Push -> B
- SW13: renamed from SW7; value SW_Push -> A
- SW2: value SW_Push -> LT1
- SW3: value SW_Push -> LT2
- SW4: value SW_Push -> RT1
- SW5: value SW_Push -> RT2
- SW6: renamed from SW12; value SW_Push -> SEL; footprint gamerino:B3W-1050 -> gamerino:TL1105-T
- SW7: renamed from SW10; value SW_Push -> START; footprint gamerino:B3W-1050 -> gamerino:TL1105-T
- SW8: renamed from SW6; value SW_Push -> BACK; footprint gamerino:B3W-1050 -> gamerino:TL1105-T
- SW9: value SW_Push -> HOME
- moved J2 81.9 mm to (95.5, 103.5)
- moved J3 81.8 mm to (180.5, 103.5)
- moved C3 16.6 mm to (127.5, 93.2), turned to 180 degrees
- moved X1 13.2 mm to (127.5, 95.5), turned to 90 degrees
- moved C4 9.84 mm to (127.5, 97.8), turned to 180 degrees
- moved SW3 3.00 mm to (103.5, 59.0)
- moved SW5 3.00 mm to (172.5, 59.0)
- moved C10 1.52 mm to (127.8, 92.0)
- moved R3 1.52 mm to (127.8, 90.5)
- moved R5 1.50 mm to (142.0, 104.5)
- moved SW10 1.00 mm to (147.0, 78.0)
- moved SW8 1.00 mm to (129.0, 78.0)
- moved C2 0.79 mm to (151.2, 63.2)
- moved C5 0.75 mm to (150.5, 65.2)
- moved C6 0.75 mm to (150.5, 66.8)
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Connections:
- R4 pad 1: Net-(D1-Pad2) -> +3V3
- R4 pad 2: +3V3 -> Net-(R4-Pad2)
- SW10 pad 1: /Y -> /OPTIONS
- SW11 pad 1: /CLEAR -> /X
- SW12 pad 1: /X -> /B
- SW13 pad 1: /START -> /A
- SW2 pad 1: GND -> /LT1
- SW2 pad 2: /LT1 -> GND
- SW3 pad 1: GND -> /LT2
- SW3 pad 2: /LT2 -> GND
- SW4 pad 1: GND -> /RT1
- SW4 pad 2: /RT1 -> GND
- SW5 pad 1: GND -> /RT2
- SW5 pad 2: /RT2 -> GND
- SW6 pad 1: /B -> /SELECT
- SW7 pad 1: /OPTIONS -> /START
- SW8 pad 1: /SELECT -> /BACK
- SW9 pad 1: /HOME -> Net-(SW9-Pad1)
- SW9 pad 3: (no net) -> /HOME
- SW9 pad 4: (no net) -> Net-(SW9-Pad4)
- SW9 pad 5: (no net) -> GND
- SW9 pad 6: (no net) -> Net-(R4-Pad2)
- U3 pad 8: /OPTS -> /OPTIONS
Routing:
- net Net-(C1-Pad2): track 0.00 -> 6.36 mm
- net GND: track 0.00 -> 5.61 mm, vias 0 -> 9
- net /XTAL2: track 0.00 -> 1.46 mm
- net +3V3: track 0.00 -> 1.02 mm
- added copper zone on F.Cu, net +3V3
- added copper zone on F.Cu, net VBUS
- removed copper zone on F.Cu, net GND
Other:
- outline, holes or cut-outs redrawn

Commit message: Update board
Parts:
- added JOY1: RKJXU, alps:RKJXU, F.Cu at (88.0, 69.6)
- added JOY2: RKJXU, alps:RKJXU, F.Cu at (168.1, 111.4)

Commit message: Update schematics
Add LHOME net
Connections:
- SW9 pad 5: GND -> LHOME
- U2 pad 31: /PC6 -> LHOME
Changed lines of the file:
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@@
-(kicad_pcb (version 20171130) (host pcbnew "(5.1.9)-1")
+(kicad_pcb (version 20171130) (host pcbnew "(5.1.5)-3")
   (general
     (thickness 1.6)
@@
     (zones 0)
     (modules 51)
-    (nets 64)
+    (nets 65)
   )
   (page A4)
@@
   (layers
     (0 F.Cu signal)
-    (31 B.Cu signal hide)
-    (34 B.Paste user hide)
+    (31 B.Cu signal)
+    (34 B.Paste user)
     (35 F.Paste user)
-    (36 B.SilkS user hide)
+    (36 B.SilkS user)
     (37 F.SilkS user)
-    (38 B.Mask user hide)
+    (38 B.Mask user)
     (39 F.Mask user)
-    (40 Dwgs.User user hide)
-    (41 Cmts.User user hide)
+    (40 Dwgs.User user)
+    (41 Cmts.User user)
     (44 Edge.Cuts user)
-    (45 Margin user hide)
-    (46 B.CrtYd user hide)
+    (45 Margin user)
+    (46 B.CrtYd user)
     (47 F.CrtYd user)
-    (48 B.Fab user hide)
+    (48 B.Fab user)
     (49 F.Fab user)
   )
@@
     (mod_text_size 1 1)
     (mod_text_width 0.15)
-    (pad_size 2 2)
-    (pad_drill 1)
+    (pad_size 1.475 0.55)
+    (pad_drill 0)
     (pad_to_mask_clearance 0.051)
     (solder_mask_min_width 0.25)
@@
   (net 62 "Net-(SW9-Pad1)")
   (net 63 "Net-(SW9-Pad4)")
+  (net 64 LHOME)
   (net_class Default "This is the default net class."
     (clearance 0.2)
@@
     (add_net /Y)
     (add_net GND)
+    (add_net LHOME)
     (add_net "Net-(C1-Pad2)")
     (add_net "Net-(C7-Pad2)")
@@
       (effects (font (size 1 1) (thickness 0.15)))
     )
-    (fp_text value RKJXU (at 7.8 8 180) (layer F.Fab)
+    (fp_text value RKJXU (at 7.8 8 180) (layer F.SilkS) hide
       (effects (font (size 1 1) (thickness 0.15)))
     )
@@
       (effects (font (size 1 1) (thickness 0.15)))
     )
-    (fp_text value RKJXU (at 7.8 8) (layer F.Fab)
+    (fp_text value RKJXU (at 7.8 8) (layer F.SilkS) hide
       (effects (font (size 1 1) (thickness 0.15)))
     )
@@
       (effects (font (size 1 1) (thickness 0.15)))
     )
-    (fp_text value MountingHole_1.5mm (at 0 3.1) (layer F.Fab)
+    (fp_text value MountingHole_1.5mm (at 0 3.1) (layer F.Fab) hide
       (effects (font (size 1 1) (thickness 0.15)))
     )
@@
       (effects (font (size 1 1) (thickness 0.15)))
     )
-    (fp_text value MountingHole_2mm (at 0 3.1) (layer F.Fab)
+    (fp_text value MountingHole_2mm (at 0 3.1) (layer F.Fab) hide
       (effects (font (size 1 1) (thickness 0.15)))
     )
@@
       (effects (font (size 1 1) (thickness 0.15)))
     )
-    (fp_text value MountingHole_1.5mm (at 0 3.1) (layer F.Fab)
+    (fp_text value MountingHole_1.5mm (at 0 3.1) (layer F.Fab) hide
       (effects (font (size 1 1) (thickness 0.15)))
     )
@@
       (effects (font (size 1 1) (thickness 0.15)))
     )
-    (fp_text value MountingHole_2mm (at 0 3.1) (layer F.Fab)
+    (fp_text value MountingHole_2mm (at 0 3.1) (layer F.Fab) hide
       (effects (font (size 1 1) (thickness 0.15)))
     )
@@
       (effects (font (size 1 1) (thickness 0.15)))
     )
-    (fp_text value USB_B_Micro (at 0 3.765165 180) (layer F.Fab)
-      (effects (font (size 1.001378 1.001378) (thickness 0.015)))
+    (fp_text value USB_B_Micro (at 0 4 180) (layer F.Fab) hide
+      (effects (font (size 1 1) (thickness 0.15)))
     )
     (fp_line (start -3.75 -2.85) (end -3.75 1.45) (layer F.Fab) (width 0.127))
@@
     (fp_line (start -3.75 1.45) (end 3.75 1.45) (layer F.Fab) (width 0.127))
     (fp_circle (center -1.3 -3.148) (end -1.2 -3.148) (layer F.Fab) (width 0.2))
-    (fp_text user PCB~EDGE (at -1.14399 2.02575 180) (layer F.Fab)
-      (effects (font (size 0.320276 0.320276) (thickness 0.015)))
+    (fp_text user PCB~EDGE (at -2 2 180) (layer F.Fab) hide
+      (effects (font (size 0.3 0.3) (thickness 0.075)))
     )
     (pad 1 smd rect (at -1.3 -2.675 180) (size 0.4 1.35) (layers F.Cu F.Paste F.Mask)
@@
       (net 28 /PB6))
     (pad 31 smd roundrect (at 5.6625 -2.4 270) (size 1.475 0.55) (layers F.Cu F.Paste F.Mask) (roundrect_rratio 0.25)
-      (net 22 /PC6))
+      (net 64 LHOME))
     (pad 32 smd roundrect (at 5.6625 -3.2 270) (size 1.475 0.55) (layers F.Cu F.Paste F.Mask) (roundrect_rratio 0.25)
       (net 20 /PC7))
@@
       (net 63 "Net-(SW9-Pad4)"))
     (pad 5 thru_hole circle (at 0 -2.54 90) (size 2 2) (drill 1) (layers *.Cu *.Mask)
-      (net 1 GND))
+      (net 64 LHOME))
     (pad 6 thru_hole circle (at 0 2.54 90) (size 2 2) (drill 1) (layers *.Cu *.Mask)
       (net 60 "Net-(R4-Pad2)"))
@@
     (connect_pads (clearance 0.508))
     (min_thickness 0.254)
-    (fill yes (arc_segments 32) (thermal_gap 0.508) (thermal_bridge_width 0.508))
+    (fill (arc_segments 32) (thermal_gap 0.508) (thermal_bridge_width 0.508))
     (polygon
       (pts
@@
     (connect_pads (clearance 0.254))
     (min_thickness 0.254)
-    (fill yes (arc_segments 32) (thermal_gap 0.254) (thermal_bridge_width 0.508))
+    (fill (arc_segments 32) (thermal_gap 0.254) (thermal_bridge_width 0.508))
     (polygon
       (pts
@@
     (connect_pads yes (clearance 0.254))
     (min_thickness 0.254)
-    (fill yes (arc_segments 32) (thermal_gap 0.254) (thermal_bridge_width 0.508))
+    (fill (arc_segments 32) (thermal_gap 0.254) (thermal_bridge_width 0.508))
     (polygon
       (pts

Commit message: Update Layout
Parts:
- added hA: M3, MountingHole:MountingHole_3.2mm_M3, F.Cu at (85.0, 63.5)
- added hB: M3, MountingHole:MountingHole_3.2mm_M3, F.Cu at (191.0, 63.5)
- added hC: M3, MountingHole:MountingHole_3.2mm_M3, F.Cu at (191.0, 107.5)
- added hD: M3, MountingHole:MountingHole_3.2mm_M3, F.Cu at (85.0, 107.5)
- C1, C10, C2, C3, C4, C5, C6, C7, C8, C9, F1, J1, R3, R5, U1, U2, X1: moved to B.Cu
- R1, R2: footprint Resistor_SMD:R_0603_1608Metric -> Resistor_SMD:R_0402_1005Metric; moved to B.Cu
- R4: moved to F.Cu
- SW10: value OPTS -> TL6210; footprint gamerino:TL1105-T -> gamerino:TL6210
- SW6: value SEL -> TL6210; footprint gamerino:TL1105-T -> gamerino:TL6210
- SW7: footprint gamerino:TL1105-T -> gamerino:TL6210
- SW8: value BACK -> TL6210; footprint gamerino:TL1105-T -> gamerino:TL6210
- SW9: value HOME -> TL3265; footprint gamerino:TL1220 -> gamerino:TL3265
- h1, h4: value MountingHole_2mm -> 2mm
- h2, h3: value MountingHole_1.5mm -> 1.5mm
- moved C3 27.9 mm to (148.8, 75.2), turned to 0 degrees
- moved C4 27.9 mm to (148.8, 79.7), turned to 0 degrees
- moved X1 27.9 mm to (148.8, 77.5)
- moved C10 27.5 mm to (148.6, 74.0), turned to 180 degrees
- moved R3 27.5 mm to (148.6, 72.5), turned to 0 degrees
- moved C2 26.5 mm to (124.8, 63.2), turned to 0 degrees
- moved C5 25.0 mm to (125.5, 65.2), turned to 180 degrees
- moved C6 25.0 mm to (125.5, 66.8), turned to 180 degrees
- moved C7 24.0 mm to (131.1, 75.6), turned to 0 degrees
- moved R5 18.3 mm to (135.7, 87.3)
- moved U1 18.0 mm to (129.0, 65.0), turned to 180 degrees
- moved U2 17.1 mm to (139.7, 78.0)
- moved C8 15.6 mm to (139.8, 69.5)
- moved C9 15.5 mm to (141.2, 69.5)
- moved C1 12.0 mm to (132.0, 65.0)
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Connections:
- net Net-(R1-Pad1) renamed D+
- net Net-(R2-Pad1) renamed D-
- SW10 pad 2: GND -> (no net)
- SW10 pad 3: (no net) -> GND
- SW6 pad 2: GND -> (no net)
- SW6 pad 3: (no net) -> GND
- SW8 pad 2: GND -> (no net)
- SW8 pad 3: (no net) -> GND
Routing:
- net D+: track 0.00 -> 2.84 mm
- net D-: track 0.00 -> 2.82 mm
- net VBUS: track 0.00 -> 2.36 mm
- net Net-(C8-Pad2): track 0.00 -> 2.07 mm
- net GND: track 5.61 -> 4.00 mm, vias 9 -> 8
- net +3V3: track 1.02 -> 0.00 mm
- added copper zone on B.Cu, net +3V3
- added copper zone on B.Cu, net VBUS
- removed copper zone on F.Cu, net VBUS
Other:
- outline, holes or cut-outs redrawn
- net class USB90 added: clearance 0.15, trace_width 0.45, via_dia 0.8, via_drill 0.4

Commit message: Update gamerino.kicad_pcb
Parts:
- U3: value TCA9539 -> TCA6416A
Connections:
- U3 pad 2: GND -> +3V3

Commit message: Routing
Parts:
- SW10: value TL6210 -> OPTS
- SW6: value TL6210 -> SEL
- SW8: value TL6210 -> CLEAR
- moved J2 46.0 mm to (110.5, 60.0), turned to 270 degrees
- moved P3 45.7 mm to (151.0, 65.5), turned to 90 degrees
- moved J3 45.7 mm to (166.5, 60.0), turned to 270 degrees
- moved R8 24.5 mm to (153.2, 78.8)
- moved R6 24.0 mm to (152.2, 82.2), turned to 180 degrees
- moved U3 21.9 mm to (157.8, 84.5)
- moved R9 18.8 mm to (159.8, 79.2), turned to 0 degrees
- moved R7 18.3 mm to (159.8, 77.5), turned to 180 degrees
- moved R4 9.95 mm to (142.4, 81.5), turned to 90 degrees
- moved C10 7.96 mm to (154.9, 78.8), turned to 270 degrees
- moved R5 2.48 mm to (134.0, 85.5)
- moved R3 1.41 mm to (147.2, 73.0), turned to 90 degrees
- moved C3 0.15 mm to (148.8, 75.3)
- moved C4 0.15 mm to (148.8, 79.8)
- moved X1 0.12 mm to (148.8, 77.6)
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Connections:
- C3 pad 1: /XTAL1 -> /XTAL2
- C4 pad 1: /XTAL2 -> /XTAL1
- P4 pad 10: /PB6 -> (no net)
- P4 pad 11: /PD4 -> /PD6
- P4 pad 12: /PB5 -> (no net)
- P4 pad 13: /PD3 -> /PD4
- P4 pad 14: /PB4 -> (no net)
- P4 pad 15: /PD2 -> /PD5
- P4 pad 3: /PE6 -> /PB6
- P4 pad 4: /PC6 -> (no net)
- P4 pad 5: /PD7 -> /PB5
- P4 pad 6: Net-(P4-Pad6) -> (no net)
- P4 pad 7: /PD6 -> /PB4
- P4 pad 8: /PB7 -> (no net)
- P4 pad 9: /PD5 -> /PD7
- SW8 pad 1: /BACK -> /CLEAR
- U2 pad 12: /PB7 -> /IRQ
- U2 pad 8: /IRQ -> (no net)
- U3 pad 10: /B -> /HS
- U3 pad 11: /A -> /LT1
- U3 pad 13: /Y -> /HE
- U3 pad 17: /HE -> /HOME
- U3 pad 18: /HS -> /CLEAR
- U3 pad 19: /LT1 -> /SELECT
- U3 pad 20: /RT1 -> /OPTIONS
- U3 pad 4: /SELECT -> /START
- U3 pad 5: /START -> /X
- U3 pad 6: /CLEAR -> /Y
- U3 pad 7: /HOME -> /RT1
- U3 pad 8: /OPTIONS -> /B
- U3 pad 9: /X -> /A
- X1 pad 1: /XTAL2 -> /XTAL1
- X1 pad 2: /XTAL1 -> /XTAL2
Routing:
- net /LT1: track 0.00 -> 112.5 mm, vias 0 -> 3
- net /RT2: track 0.00 -> 91.2 mm, vias 0 -> 3
- net /J1X: track 0.00 -> 76.3 mm, vias 0 -> 3
- net /J1Y: track 0.00 -> 73.1 mm, vias 0 -> 3
- net /HS: track 0.00 -> 71.5 mm, vias 0 -> 3
- net /SELECT: track 0.00 -> 70.7 mm, vias 0 -> 3
- net /J2X: track 0.00 -> 68.7 mm, vias 0 -> 1
- net /J2Y: track 0.00 -> 67.0 mm, vias 0 -> 1
- net /HW: track 0.00 -> 59.3 mm, vias 0 -> 3
- net /LT2: track 0.00 -> 54.7 mm, vias 0 -> 1
- net /HP: track 0.00 -> 51.6 mm, vias 0 -> 3
- net /HN: track 0.00 -> 49.4 mm, vias 0 -> 3
- net /HE: track 0.00 -> 47.3 mm, vias 0 -> 3
- net /RT1: track 0.00 -> 45.4 mm
- net /CLEAR: track 0.00 -> 40.0 mm, vias 0 -> 3
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