File: PCB/gamerino.kicad_pcb (KiCad board)
At the start: 2 copper layers, 125 x 63 mm, 76 parts, among them J1 USB_B_Micro, J2 LT2, J3 RT2, J4 ACT2, J5 ACT2, P1 JOY1, P2 JOY2, P3 ICSP, P4 AUX, Q1 DMN601WK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

Commit message: Update
Parts:
- added U4: ESDS304, Package_TO_SOT_SMD:SOT-23-5, F.Cu at (137.7, 67.9)
Routing:
- net GND: track 7.30 -> 11.2 mm, vias 8 -> 9
- net D-: track 2.82 -> 4.58 mm, vias 0 -> 1
- net D+: track 2.84 -> 4.57 mm, vias 0 -> 1
- net VBUS: track 7.98 -> 8.93 mm, vias 0 -> 1
- net /SCK: track 12.0 -> 11.4 mm
- net /MOSI: track 13.0 -> 12.4 mm
Other:
- rule via_min_drill: 0.3 -> 0.2
- rule via_min_size: 0.4 -> 0.5

Commit message: Update
Parts:
- removed the LOGO2 at (94.0, 94.0)
- added LOGO0: LOGO-Gamerino, gamerino:gamerino_logo, B.Cu at (94.0, 94.0)
- added REF**: RKJXV1224, gamerino:RKJXV1224, F.Cu at (95.0, 79.0)
- renumbered U4 to D7
Connections:
- D7 pad 1: (no net) -> Net-(D7-Pad1)
Routing:
- net /A: track 26.3 -> 19.6 mm
- removed copper zone on B.Cu, net /RT2

Commit message: Update
Parts:
- removed REF**: RKJXV1224, gamerino:RKJXV1224

Commit message: Update to KiCAD 8.0
Update to KiCAD 8.0
Other:
- net class Default removed
- net class USB90 removed
